File: regius.sch (KiCad schematic (older format))
At the start: 56 parts, among them J1 Conn_01x02, J7 Conn_01x02, SW1 Reset, U5 LM1117-3.3

Commit message: add footprints
Parts:
- added J10: A10, Connector_PinHeader_2.54mm:PinHeader_1x02_P2.54mm_Vertical, symbol Connector_Generic:Conn_01x02
- added J11: A9, Connector_PinHeader_2.54mm:PinHeader_1x02_P2.54mm_Vertical, symbol Connector_Generic:Conn_01x02
- added J12: A8, Connector_PinHeader_2.54mm:PinHeader_1x02_P2.54mm_Vertical, symbol Connector_Generic:Conn_01x02
- added J13: A7, Connector_PinHeader_2.54mm:PinHeader_1x02_P2.54mm_Vertical, symbol Connector_Generic:Conn_01x02
- added J14: A6, Connector_PinHeader_2.54mm:PinHeader_1x02_P2.54mm_Vertical, symbol Connector_Generic:Conn_01x02
- added J15: A5, Connector_PinHeader_2.54mm:PinHeader_1x02_P2.54mm_Vertical, symbol Connector_Generic:Conn_01x02
- added J16: A4, Connector_PinHeader_2.54mm:PinHeader_1x02_P2.54mm_Vertical, symbol Connector_Generic:Conn_01x02
- added J17: A3, Connector_PinHeader_2.54mm:PinHeader_1x02_P2.54mm_Vertical, symbol Connector_Generic:Conn_01x02
- added J18: A2, Connector_PinHeader_2.54mm:PinHeader_1x02_P2.54mm_Vertical, symbol Connector_Generic:Conn_01x02
- added J19: D28, Connector_PinHeader_2.54mm:PinHeader_1x02_P2.54mm_Vertical, symbol Connector_Generic:Conn_01x02
- added J2: D3, Connector_PinHeader_2.54mm:PinHeader_1x02_P2.54mm_Vertical, symbol Connector_Generic:Conn_01x02
- added J20: D27, Connector_PinHeader_2.54mm:PinHeader_1x02_P2.54mm_Vertical, symbol Connector_Generic:Conn_01x02
- added J21: D26, Connector_PinHeader_2.54mm:PinHeader_1x02_P2.54mm_Vertical, symbol Connector_Generic:Conn_01x02
- added J22: D25, Connector_PinHeader_2.54mm:PinHeader_1x02_P2.54mm_Vertical, symbol Connector_Generic:Conn_01x02
- added J23: D24, Connector_PinHeader_2.54mm:PinHeader_1x02_P2.54mm_Vertical, symbol Connector_Generic:Conn_01x02
- added J24: D23, Connector_PinHeader_2.54mm:PinHeader_1x02_P2.54mm_Vertical, symbol Connector_Generic:Conn_01x02
- added J25: D22, Connector_PinHeader_2.54mm:PinHeader_1x02_P2.54mm_Vertical, symbol Connector_Generic:Conn_01x02
- added J26: D12, Connector_PinHeader_2.54mm:PinHeader_1x02_P2.54mm_Vertical, symbol Connector_Generic:Conn_01x02
- added J27: D11, Connector_PinHeader_2.54mm:PinHeader_1x02_P2.54mm_Vertical, symbol Connector_Generic:Conn_01x02
- added J28: D10, Connector_PinHeader_2.54mm:PinHeader_1x02_P2.54mm_Vertical, symbol Connector_Generic:Conn_01x02
- added J29: D9, Connector_PinHeader_2.54mm:PinHeader_1x02_P2.54mm_Vertical, symbol Connector_Generic:Conn_01x02
- added J3: D2, Connector_PinHeader_2.54mm:PinHeader_1x02_P2.54mm_Vertical, symbol Connector_Generic:Conn_01x02
- added J30: D8, Connector_PinHeader_2.54mm:PinHeader_1x02_P2.54mm_Vertical, symbol Connector_Generic:Conn_01x02
- added J31: D7, Connector_PinHeader_2.54mm:PinHeader_1x02_P2.54mm_Vertical, symbol Connector_Generic:Conn_01x02
- added J32: D6, Connector_PinHeader_2.54mm:PinHeader_1x02_P2.54mm_Vertical, symbol Connector_Generic:Conn_01x02
- added J33: D5, Connector_PinHeader_2.54mm:PinHeader_1x02_P2.54mm_Vertical, symbol Connector_Generic:Conn_01x02
- added J34: D4, Connector_PinHeader_2.54mm:PinHeader_1x02_P2.54mm_Vertical, symbol Connector_Generic:Conn_01x02
- added J35: D44, Connector_PinHeader_2.54mm:PinHeader_1x02_P2.54mm_Vertical, symbol Connector_Generic:Conn_01x02
- added J36: D43, Connector_PinHeader_2.54mm:PinHeader_1x02_P2.54mm_Vertical, symbol Connector_Generic:Conn_01x02
- added J37: D42, Connector_PinHeader_2.54mm:PinHeader_1x02_P2.54mm_Vertical, symbol Connector_Generic:Conn_01x02
- added J38: D41, Connector_PinHeader_2.54mm:PinHeader_1x02_P2.54mm_Vertical, symbol Connector_Generic:Conn_01x02
- added J39: D40, Connector_PinHeader_2.54mm:PinHeader_1x02_P2.54mm_Vertical, symbol Connector_Generic:Conn_01x02
- added J4: A15, Connector_PinHeader_2.54mm:PinHeader_1x02_P2.54mm_Vertical, symbol Connector_Generic:Conn_01x02
- added J40: D39, Connector_PinHeader_2.54mm:PinHeader_1x02_P2.54mm_Vertical, symbol Connector_Generic:Conn_01x02
- added J41: D38, Connector_PinHeader_2.54mm:PinHeader_1x02_P2.54mm_Vertical, symbol Connector_Generic:Conn_01x02
- added J42: D37, Connector_PinHeader_2.54mm:PinHeader_1x02_P2.54mm_Vertical, symbol Connector_Generic:Conn_01x02
- added J43: D36, Connector_PinHeader_2.54mm:PinHeader_1x02_P2.54mm_Vertical, symbol Connector_Generic:Conn_01x02
- added J44: D35, Connector_PinHeader_2.54mm:PinHeader_1x02_P2.54mm_Vertical, symbol Connector_Generic:Conn_01x02
- added J45: D34, Connector_PinHeader_2.54mm:PinHeader_1x02_P2.54mm_Vertical, symbol Connector_Generic:Conn_01x02
- added J46: D33, Connector_PinHeader_2.54mm:PinHeader_1x02_P2.54mm_Vertical, symbol Connector_Generic:Conn_01x02
- added J47: D32, Connector_PinHeader_2.54mm:PinHeader_1x02_P2.54mm_Vertical, symbol Connector_Generic:Conn_01x02
- added J48: D31, Connector_PinHeader_2.54mm:PinHeader_1x02_P2.54mm_Vertical, symbol Connector_Generic:Conn_01x02
- added J49: D30, Connector_PinHeader_2.54mm:PinHeader_1x02_P2.54mm_Vertical, symbol Connector_Generic:Conn_01x02
- added J5: A14, Connector_PinHeader_2.54mm:PinHeader_1x02_P2.54mm_Vertical, symbol Connector_Generic:Conn_01x02
- added J50: D29, Connector_PinHeader_2.54mm:PinHeader_1x02_P2.54mm_Vertical, symbol Connector_Generic:Conn_01x02
- added J51: D19, Connector_PinHeader_2.54mm:PinHeader_1x02_P2.54mm_Vertical, symbol Connector_Generic:Conn_01x02
- added J52: D18, Connector_PinHeader_2.54mm:PinHeader_1x02_P2.54mm_Vertical, symbol Connector_Generic:Conn_01x02
- added J53: D17, Connector_PinHeader_2.54mm:PinHeader_1x02_P2.54mm_Vertical, symbol Connector_Generic:Conn_01x02
- added J54: D16, Connector_PinHeader_2.54mm:PinHeader_1x02_P2.54mm_Vertical, symbol Connector_Generic:Conn_01x02
- added J55: D15, Connector_PinHeader_2.54mm:PinHeader_1x02_P2.54mm_Vertical, symbol Connector_Generic:Conn_01x02
- added J56: D14, Connector_PinHeader_2.54mm:PinHeader_1x02_P2.54mm_Vertical, symbol Connector_Generic:Conn_01x02
- added J57: D52, Connector_PinHeader_2.54mm:PinHeader_1x02_P2.54mm_Vertical, symbol Connector_Generic:Conn_01x02
- added J58: D50, Connector_PinHeader_2.54mm:PinHeader_1x02_P2.54mm_Vertical, symbol Connector_Generic:Conn_01x02
- added J59: D49, Connector_PinHeader_2.54mm:PinHeader_1x02_P2.54mm_Vertical, symbol Connector_Generic:Conn_01x02
- added J6: A13, Connector_PinHeader_2.54mm:PinHeader_1x02_P2.54mm_Vertical, symbol Connector_Generic:Conn_01x02
- added J60: D48, Connector_PinHeader_2.54mm:PinHeader_1x02_P2.54mm_Vertical, symbol Connector_Generic:Conn_01x02
- added J61: D47, Connector_PinHeader_2.54mm:PinHeader_1x02_P2.54mm_Vertical, symbol Connector_Generic:Conn_01x02
- added J62: D46, Connector_PinHeader_2.54mm:PinHeader_1x02_P2.54mm_Vertical, symbol Connector_Generic:Conn_01x02
- added J63: D45, Connector_PinHeader_2.54mm:PinHeader_1x02_P2.54mm_Vertical, symbol Connector_Generic:Conn_01x02
- added J69: 4WIRELED, Connector_PinHeader_2.54mm:PinHeader_1x02_P2.54mm_Vertical, symbol Connector_Generic:Conn_01x02
- added J8: A12, Connector_PinHeader_2.54mm:PinHeader_1x02_P2.54mm_Vertical, symbol Connector_Generic:Conn_01x02
- added J9: A11, Connector_PinHeader_2.54mm:PinHeader_1x02_P2.54mm_Vertical, symbol Connector_Generic:Conn_01x02
- C1, C11, C12, C13, C14, C15, C16, C17, C18, C19, C2, C20, C3, C4, C5, C6, C7: renamed from C?; footprint (none) -> Capacitor_SMD:C_0603_1608Metric
- D1, D2, D3: renamed from D?; footprint (none) -> LED_SMD:LED_0603_1608Metric
- FB1: renamed from FB?; footprint (none) -> Inductor_SMD:L_0603_1608Metric
- J1: value Conn_01x02 -> 3.3v
- J64, J65, J66, J68, J70, J72, J73: renamed from J?; footprint (none) -> Connector_PinHeader_2.54mm:PinHeader_1x02_P2.54mm_Vertical
- J67: renamed from J?; footprint (none) -> Connector_PinHeader_1.27mm:PinHeader_2x05_P1.27mm_Vertical
- J7: value Conn_01x02 -> VCC
- J71: renamed from J?; footprint (none) -> Connector_Card:microSD_HC_Hirose_DM3D-SF
- J74: renamed from J?; footprint (none) -> Connector_USB:USB_Micro-B_Amphenol_10103594-0001LF_Horizontal
- U2: renamed from U?; footprint (none) -> Package_QFP:TQFP-128_14x14mm_P0.4mm
- Y1: renamed from Y?; footprint (none) -> Crystal:Crystal_SMD_3215-2Pin_3.2x1.5mm
- gave numbers to parts that had none: 8
Connections:
- net A10: now also J10.1 (Pin_1)
- net A11: now also J9.1 (Pin_1)
- net A12: now also J8.1 (Pin_1)
- net A13: now also J6.1 (Pin_1)
- net A14: now also J5.1 (Pin_1)
- net A15: now also J4.1 (Pin_1)
- net A2: now also J18.1 (Pin_1)
- net A3: now also J17.1 (Pin_1)
- net A4: now also J16.1 (Pin_1)
- net A5: now also J15.1 (Pin_1)
- net A6: now also J14.1 (Pin_1)
- net A7: now also J13.1 (Pin_1)
- net A8: now also J12.1 (Pin_1)
- net A9: now also J11.1 (Pin_1)
- net D10: now also J28.1 (Pin_1)
- net D11: now also J27.1 (Pin_1)
- net D12: now also J26.1 (Pin_1)
- net D2: now also J3.1 (Pin_1)
- net D22: now also J25.1 (Pin_1)
- net D23: now also J24.1 (Pin_1)
- net D26: now also J21.1 (Pin_1)
- net D27: now also J20.1 (Pin_1)
- net D28: now also J19.1 (Pin_1)
- net D29: now also J50.1 (Pin_1)
- net D3: now also J2.1 (Pin_1)
- net D30: now also J49.1 (Pin_1)
- net D31: now also J48.1 (Pin_1)
- net D32: now also J47.1 (Pin_1)
- net D4: now also J34.1 (Pin_1)
- net D5: now also J33.1 (Pin_1)
- net D6: now also J32.1 (Pin_1)
- net D7: now also J31.1 (Pin_1)
- net D8: now also J30.1 (Pin_1)
- net D9: now also J29.1 (Pin_1)
- net GND: now also J10.2 (Pin_2), J11.2 (Pin_2), J12.2 (Pin_2), J13.2 (Pin_2), J14.2 (Pin_2), J15.2 (Pin_2), J16.2 (Pin_2), J17.2 (Pin_2), J18.2 (Pin_2), J19.2 (Pin_2), J2.2 (Pin_2), J20.2 (Pin_2), J21.2 (Pin_2), J22.2 (Pin_2), J23.2 (Pin_2), J24.2 (Pin_2), J25.2 (Pin_2), J26.2 (Pin_2), J27.2 (Pin_2), J28.2 (Pin_2), J29.2 (Pin_2), J3.2 (Pin_2), J30.2 (Pin_2), J31.2 (Pin_2), J32.2 (Pin_2), J33.2 (Pin_2), J34.2 (Pin_2), J35.2 (Pin_2), J36.2 (Pin_2), J37.2 (Pin_2), J38.2 (Pin_2), J39.2 (Pin_2), J4.2 (Pin_2), J40.2 (Pin_2), J41.2 (Pin_2), J42.2 (Pin_2), J43.2 (Pin_2), J44.2 (Pin_2), J45.2 (Pin_2), J46.2 (Pin_2), J47.2 (Pin_2), J48.2 (Pin_2), J49.2 (Pin_2), J5.2 (Pin_2), J50.2 (Pin_2), J51.2 (Pin_2), J52.2 (Pin_2), J53.2 (Pin_2), J54.2 (Pin_2), J55.2 (Pin_2), J56.2 (Pin_2), J57.2 (Pin_2), J58.2 (Pin_2), J59.2 (Pin_2), J6.2 (Pin_2), J60.2 (Pin_2), J61.2 (Pin_2), J62.2 (Pin_2), J63.2 (Pin_2), J8.2 (Pin_2), J9.2 (Pin_2)
- net D48: now reaches U2.27 (PC04)
- net D48: now also J60.1 (Pin_1)
- net D49: now reaches U2.28 (PC05)
- net D49: now also J59.1 (Pin_1)
- net D46: now reaches U2.29 (PC06)
- net D46: now also J62.1 (Pin_1)
- net D47: now reaches U2.30 (PC07)
- net D47: now also J61.1 (Pin_1)
- net D39: now reaches U2.43 (PB14)
- net D39: now also J40.1 (Pin_1)
- net D38: now reaches U2.44 (PB15)
- net D38: now also J41.1 (Pin_1)
- net at U2.47 (PD08): now also J69.2 (Pin_2)
- net at U2.48 (PD09): now also J69.1 (Pin_1)
- net D45: now reaches U2.52 (PC10)
- net D45: now also J63.1 (Pin_1)
- net D44: now reaches U2.55 (PC11)
- net D44: now also J35.1 (Pin_1)
- net D41: now reaches U2.56 (PC12)
- net D41: now also J38.1 (Pin_1)
- net D40: now reaches U2.57 (PC13)
- net D40: now also J39.1 (Pin_1)
- net D43: now reaches U2.58 (PC14)
- net D43: now also J36.1 (Pin_1)
- net D42: now reaches U2.59 (PC15)
- net D42: now also J37.1 (Pin_1)
- net D37: now reaches U2.66 (PA16)
- net D37: now also J42.1 (Pin_1)
- net D36: now reaches U2.67 (PA17)
- net D36: now also J43.1 (Pin_1)
- net D35: now reaches U2.68 (PA18)
- net D35: now also J44.1 (Pin_1)
- net D34: now reaches U2.69 (PA19)
- net D34: now also J45.1 (Pin_1)
- net D33: now reaches U2.88 (PA20)
- net D33: now also J46.1 (Pin_1)
- new net D14: J56.1 (Pin_1)
- new net D15: J55.1 (Pin_1)
- new net D16: J54.1 (Pin_1)
- new net D17: J53.1 (Pin_1)
- new net D18: J52.1 (Pin_1)
- new net D19: J51.1 (Pin_1)
- new net D24: J23.1 (Pin_1)
- new net D25: J22.1 (Pin_1)
- new net D50: J58.1 (Pin_1)
- new net D52: J57.1 (Pin_1)
Other:
- moved on the sheet: H1, H2, H3, H4, H5, H6, H8

Commit message: add 3d image
Parts:
- U1: footprint SOIC127P600X175-8N -> (none)
Other:
- moved on the sheet: C1, C10, C11, C12, C13, C14, C15, C16, C17, C18, C19, C2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

Commit message: update schematic tca9548
Parts:
- removed H1, H6, H8: MountingHole, MountingHole:MountingHole_3mm, symbol Mechanical:MountingHole
- removed J40: D39, Connector_PinHeader_2.54mm:PinHeader_1x02_P2.54mm_Vertical, symbol Connector_Generic:Conn_01x02
- added C21: C_Small, Capacitor_SMD:C_0603_1608Metric, symbol Device:C_Small
- added D6: LED_Small, LED_SMD:LED_0603_1608Metric, symbol Device:LED_Small
- added J40: CAN, Connector_PinHeader_2.54mm:PinHeader_1x02_P2.54mm_Vertical, symbol Connector_Generic:Conn_01x03
- added J75, J76, J77, J78, J79, J80: I2C, Connector_PinHeader_2.54mm:PinHeader_1x02_P2.54mm_Vertical, symbol Connector_Generic:Conn_01x02
- added JP1, JP2, JP3: SolderJumper_2_Open, Jumper:SolderJumper-2_P1.3mm_Open_RoundedPad1.0x1.5mm, symbol Jumper:SolderJumper_2_Open
- added R10, R11, R12, R7, R8, R9: R10K, Resistor_SMD:R_0603_1608Metric, symbol Device:R
- added R13: R1K, Resistor_SMD:R_0603_1608Metric, symbol Device:R
- added U3: TCA9548APWR, Package_SO:TSSOP-24_4.4x7.8mm_P0.65mm, symbol Interface_Expansion:TCA9548APWR
- J41: value D38 -> I2C
- J68: value TXRX1 -> TXRX1CAN
- U1: footprint (none) -> GD25Q32CTIGR:SOIC127P600X175-8N
Connections:
- net +3V3: now also R6.1, C21.2, D6.2 (A), JP1.1 (A), JP2.1 (A), JP3.1 (A), R7.1, R8.1, R9.1, U3.24 (VCC); no longer R6.2
- net D38: now also J40.1 (Pin_1); no longer J41.1 (Pin_1)
- net D39: now also J40.2 (Pin_2)
- net GND: now also C21.1, J40.3 (Pin_3), R10.2, R11.2, R12.2, R13.2, U3.12 (GND); no longer J41.2 (Pin_2)
- net RESET: now reaches C8.1, J67.6 (Pin_6), R1.2, U2.114 (RESETN)
- net RESET: now also R6.2, R9.2, U3.3 (~RESET); no longer R6.1
- net at U2.70 (PC16): now also R7.2, U3.23 (SDA); no longer J73.2 (Pin_2)
- net at U2.71 (PC17): now also R8.2, U3.22 (SCL); no longer J73.1 (Pin_1)
- new net: J73.1 (Pin_1), U3.5 (SC0)
- new net: J73.2 (Pin_2), U3.4 (SD0)
- new net: JP3.2 (B), R12.1, U3.1 (A0)
- new net: J76.2 (Pin_2), U3.10 (SD3)
- new net: J76.1 (Pin_1), U3.11 (SC3)
- new net: J77.2 (Pin_2), U3.13 (SD4)
- new net: J77.1 (Pin_1), U3.14 (SC4)
- new net: J78.2 (Pin_2), U3.15 (SD5)
- new net: J78.1 (Pin_1), U3.16 (SC5)
- new net: J79.2 (Pin_2), U3.17 (SD6)
- new net: J79.1 (Pin_1), U3.18 (SC6)
- new net: J80.2 (Pin_2), U3.19 (SD7)
- new net: JP2.2 (B), R11.1, U3.2 (A1)
- new net: J80.1 (Pin_1), U3.20 (SC7)
- new net: JP1.2 (B), R10.1, U3.21 (A2)
- new net: J41.2 (Pin_2), U3.6 (SD1)
- new net: J41.1 (Pin_1), U3.7 (SC1)
- new net: J75.2 (Pin_2), U3.8 (SD2)
- new net: J75.1 (Pin_1), U3.9 (SC2)
- new net: D6.1 (K), R13.1
Other:
- moved on the sheet: J35, J36, J37, J38, J39, J73

Commit message: update layout design
Parts:
- removed FB1: Ferrite_Bead_Small, Inductor_SMD:L_0603_1608Metric, symbol Device:Ferrite_Bead_Small
- removed J19: D28, Connector_PinHeader_2.54mm:PinHeader_1x02_P2.54mm_Vertical, symbol Connector_Generic:Conn_01x02
- removed J22: D25, Connector_PinHeader_2.54mm:PinHeader_1x02_P2.54mm_Vertical, symbol Connector_Generic:Conn_01x02
- removed J23: D24, Connector_PinHeader_2.54mm:PinHeader_1x02_P2.54mm_Vertical, symbol Connector_Generic:Conn_01x02
- removed J51: D19, Connector_PinHeader_2.54mm:PinHeader_1x02_P2.54mm_Vertical, symbol Connector_Generic:Conn_01x02
- removed J52: D18, Connector_PinHeader_2.54mm:PinHeader_1x02_P2.54mm_Vertical, symbol Connector_Generic:Conn_01x02
- removed J53: D17, Connector_PinHeader_2.54mm:PinHeader_1x02_P2.54mm_Vertical, symbol Connector_Generic:Conn_01x02
- removed J54: D16, Connector_PinHeader_2.54mm:PinHeader_1x02_P2.54mm_Vertical, symbol Connector_Generic:Conn_01x02
- removed J55: D15, Connector_PinHeader_2.54mm:PinHeader_1x02_P2.54mm_Vertical, symbol Connector_Generic:Conn_01x02
- removed J56: D14, Connector_PinHeader_2.54mm:PinHeader_1x02_P2.54mm_Vertical, symbol Connector_Generic:Conn_01x02
- J40, J68, J70: footprint Connector_PinHeader_2.54mm:PinHeader_1x02_P2.54mm_Vertical -> Connector_PinHeader_2.54mm:PinHeader_1x03_P2.54mm_Vertical
Connections:
- net +3V3: now also C3.2, C4.2, C5.2, U2.15 (VDDANA), U2.26 (VDDANA), U2.6 (VDDANA)
- net A1: no longer names the net of J66.1 (Pin_1), U2.22 (PA05)
Changed lines of the file:
@@
 Wire Wire Line
 	16450 10650 17100 10650
-$Comp
-L Device:Ferrite_Bead_Small FB1
-U 1 1 5CCF8350
-P 15200 10050
-F 0 "FB1" H 15300 10096 50  0000 L CNN
-F 1 "Ferrite_Bead_Small" H 15300 10005 50  0000 L CNN
-F 2 "Inductor_SMD:L_0603_1608Metric" V 15130 10050 50  0001 C CNN
-F 3 "~" H 15200 10050 50  0001 C CNN
-	1    15200 10050
-	0    1    1    0
-$EndComp
 Connection ~ 16200 10050
 $Comp
@@
 	1    0    0    -1
 $EndComp
-Wire Wire Line
-	15300 10050 15800 10050
-Wire Wire Line
-	15100 10050 14700 10050
 $Comp
 L Device:Crystal Y1
@@
 Wire Wire Line
 	18000 4300 18000 3800
-Text Label 16500 9650 0    50   ~ 0
-A1
 Wire Wire Line
 	17800 7050 17800 6850
@@
 F 0 "J70" V 20566 5812 50  0000 R CNN
 F 1 "TXRX" V 20475 5812 50  0000 R CNN
-F 2 "Connector_PinHeader_2.54mm:PinHeader_1x02_P2.54mm_Vertical" H 20600 6000 50  0001 C CNN
+F 2 "Connector_PinHeader_2.54mm:PinHeader_1x03_P2.54mm_Vertical" H 20600 6000 50  0001 C CNN
 F 3 "~" H 20600 6000 50  0001 C CNN
 	1    20600 6000
@@
 F 0 "J68" V 18473 12730 50  0000 L CNN
 F 1 "TXRX1CAN" V 18564 12730 50  0000 L CNN
-F 2 "Connector_PinHeader_2.54mm:PinHeader_1x02_P2.54mm_Vertical" H 18600 12550 50  0001 C CNN
+F 2 "Connector_PinHeader_2.54mm:PinHeader_1x03_P2.54mm_Vertical" H 18600 12550 50  0001 C CNN
 F 3 "~" H 18600 12550 50  0001 C CNN
 	1    18600 12550
@@
 	19200 11150 19200 12100
 $Comp
-L Connector_Generic:Conn_01x02 J51
-U 1 1 5D2267A3
-P 11350 5700
-F 0 "J51" H 11430 5692 50  0000 L CNN
-F 1 "D19" V 11650 5450 50  0000 L CNN
-F 2 "Connector_PinHeader_2.54mm:PinHeader_1x02_P2.54mm_Vertical" H 11350 5700 50  0001 C CNN
-F 3 "~" H 11350 5700 50  0001 C CNN
-	1    11350 5700
-	-1   0    0    1
-$EndComp
-Wire Wire Line
-	11550 5600 11750 5600
-Wire Wire Line
-	11550 5700 12100 5700
-Text Label 12100 5700 0    50   ~ 0
-D19
-$Comp
-L Connector_Generic:Conn_01x02 J52
-U 1 1 5D2B4025
-P 11350 6050
-F 0 "J52" H 11430 6042 50  0000 L CNN
-F 1 "D18" V 11650 5800 50  0000 L CNN
-F 2 "Connector_PinHeader_2.54mm:PinHeader_1x02_P2.54mm_Vertical" H 11350 6050 50  0001 C CNN
-F 3 "~" H 11350 6050 50  0001 C CNN
-	1    11350 6050
-	-1   0    0    1
-$EndComp
-Wire Wire Line
-	11550 5950 11750 5950
-Wire Wire Line
-	11550 6050 12100 6050
-Text Label 12100 6050 0    50   ~ 0
-D18
-$Comp
-L Connector_Generic:Conn_01x02 J53
-U 1 1 5D2B402E
-P 11350 6400
-F 0 "J53" H 11430 6392 50  0000 L CNN
-F 1 "D17" V 11650 6150 50  0000 L CNN
-F 2 "Connector_PinHeader_2.54mm:PinHeader_1x02_P2.54mm_Vertical" H 11350 6400 50  0001 C CNN
-F 3 "~" H 11350 6400 50  0001 C CNN
-	1    11350 6400
-	-1   0    0    1
-$EndComp
-Wire Wire Line
-	11550 6300 11750 6300
-Wire Wire Line
-	11550 6400 12100 6400
-Text Label 12100 6400 0    50   ~ 0
-D17
-$Comp
-L Connector_Generic:Conn_01x02 J54
-U 1 1 5D2B4037
-P 11350 6750
-F 0 "J54" H 11430 6742 50  0000 L CNN
-F 1 "D16" V 11650 6500 50  0000 L CNN
-F 2 "Connector_PinHeader_2.54mm:PinHeader_1x02_P2.54mm_Vertical" H 11350 6750 50  0001 C CNN
-F 3 "~" H 11350 6750 50  0001 C CNN
-	1    11350 6750
-	-1   0    0    1
-$EndComp
-Wire Wire Line
-	11550 6650 11750 6650
-Wire Wire Line
-	11550 6750 12100 6750
-Text Label 12100 6750 0    50   ~ 0
-D16
-$Comp
-L Connector_Generic:Conn_01x02 J55
-U 1 1 5D2B4040
-P 11350 7100
-F 0 "J55" H 11430 7092 50  0000 L CNN
-F 1 "D15" V 11650 6850 50  0000 L CNN
-F 2 "Connector_PinHeader_2.54mm:PinHeader_1x02_P2.54mm_Vertical" H 11350 7100 50  0001 C CNN
-F 3 "~" H 11350 7100 50  0001 C CNN
-	1    11350 7100
-	-1   0    0    1
-$EndComp
-Wire Wire Line
-	11550 7000 11750 7000
-Wire Wire Line
-	11550 7100 12100 7100
-Text Label 12100 7100 0    50   ~ 0
-D15
-$Comp
-L Connector_Generic:Conn_01x02 J56
-U 1 1 5D383940
-P 11350 7450
-F 0 "J56" H 11430 7442 50  0000 L CNN
-F 1 "D14" V 11650 7200 50  0000 L CNN
-F 2 "Connector_PinHeader_2.54mm:PinHeader_1x02_P2.54mm_Vertical" H 11350 7450 50  0001 C CNN
-F 3 "~" H 11350 7450 50  0001 C CNN
-	1    11350 7450
-	-1   0    0    1
-$EndComp
-Wire Wire Line
-	11550 7350 11750 7350
-Wire Wire Line
-	11550 7450 12100 7450
-Text Label 12100 7450 0    50   ~ 0
-D14
-$Comp
 L Connector_Generic:Conn_01x02 J57
 U 1 1 5D383949
@@
 D29
 $Comp
-L Connector_Generic:Conn_01x02 J19
-U 1 1 5DF95EBD
-P 7800 4650
-F 0 "J19" H 7880 4642 50  0000 L CNN
-F 1 "D28" V 8100 4400 50  0000 L CNN
-F 2 "Connector_PinHeader_2.54mm:PinHeader_1x02_P2.54mm_Vertical" H 7800 4650 50  0001 C CNN
-F 3 "~" H 7800 4650 50  0001 C CNN
-	1    7800 4650
-	-1   0    0    1
-$EndComp
-Wire Wire Line
-	8000 4550 8200 4550
-Wire Wire Line
-	8000 4650 8550 4650
-Text Label 8550 4650 0    50   ~ 0
-D28
-$Comp
 L Connector_Generic:Conn_01x02 J20
 U 1 1 5DF95EC6
@@
 D26
 $Comp
-L Connector_Generic:Conn_01x02 J22
-U 1 1 5DF95ED8
-P 7800 5700
-F 0 "J22" H 7880 5692 50  0000 L CNN
-F 1 "D25" V 8100 5450 50  0000 L CNN
-F 2 "Connector_PinHeader_2.54mm:PinHeader_1x02_P2.54mm_Vertical" H 7800 5700 50  0001 C CNN
-F 3 "~" H 7800 5700 50  0001 C CNN
-	1    7800 5700
-	-1   0    0    1
-$EndComp
-Wire Wire Line
-	8000 5600 8200 5600
-Wire Wire Line
-	8000 5700 8550 5700
-Text Label 8550 5700 0    50   ~ 0
-D25
-$Comp
-L Connector_Generic:Conn_01x02 J23
-U 1 1 5DF95EE1
-P 7800 6050
-F 0 "J23" H 7880 6042 50  0000 L CNN
-F 1 "D24" V 8100 5800 50  0000 L CNN
-F 2 "Connector_PinHeader_2.54mm:PinHeader_1x02_P2.54mm_Vertical" H 7800 6050 50  0001 C CNN
-F 3 "~" H 7800 6050 50  0001 C CNN
-	1    7800 6050
-	-1   0    0    1
-$EndComp
-Wire Wire Line
-	8000 5950 8200 5950
-Wire Wire Line
-	8000 6050 8550 6050
-Text Label 8550 6050 0    50   ~ 0
-D24
-$Comp
 L Connector_Generic:Conn_01x02 J24
 U 1 1 5DF95EEA
@@
 Wire Wire Line
 	8000 6400 8550 6400
-Text Label 8550 6400 0    50   ~ 0
-D23
 $Comp
 L Connector_Generic:Conn_01x02 J25
@@
 Wire Wire Line
 	11750 9800 11750 9450
-Connection ~ 11750 5600
-Connection ~ 11750 5950
-Wire Wire Line
-	11750 5950 11750 5600
-Connection ~ 11750 6300
-Wire Wire Line
-	11750 6300 11750 5950
-Connection ~ 11750 6650
-Wire Wire Line
-	11750 6650 11750 6300
-Connection ~ 11750 7000
-Wire Wire Line
-	11750 7000 11750 6650
-Connection ~ 11750 7350
-Wire Wire Line
-	11750 7350 11750 7000
 Connection ~ 11750 7700
-Wire Wire Line
-	11750 7700 11750 7350
 Connection ~ 11750 8050
 Wire Wire Line
@@
 Wire Wire Line
 	8200 3950 6500 3950
-Connection ~ 8200 4550
-Wire Wire Line
-	8200 4550 8200 3950
 Connection ~ 8200 4900
-Wire Wire Line
-	8200 4900 8200 4550
 Connection ~ 8200 5250
 Wire Wire Line
 	8200 5250 8200 4900
-Connection ~ 8200 5600
-Wire Wire Line
-	8200 5600 8200 5250
-Connection ~ 8200 5950
-Wire Wire Line
-	8200 5950 8200 5600
 Connection ~ 8200 6300
-Wire Wire Line
-	8200 6300 8200 5950
 Connection ~ 8200 6650
 Wire Wire Line
@@
 Wire Wire Line
 	8200 9450 8200 9100
-Wire Wire Line
-	11750 3950 11750 5600
 Wire Wire Line
 	11750 10550 11750 9800
@@
 F 0 "J40" V 18673 13330 50  0000 L CNN
 F 1 "CAN" V 18764 13330 50  0000 L CNN
-F 2 "Connector_PinHeader_2.54mm:PinHeader_1x02_P2.54mm_Vertical" H 18800 13150 50  0001 C CNN
+F 2 "Connector_PinHeader_2.54mm:PinHeader_1x03_P2.54mm_Vertical" H 18800 13150 50  0001 C CNN
 F 3 "~" H 18800 13150 50  0001 C CNN
 	1    18800 13150
@@
 Wire Wire Line
 	25650 12150 26050 12150
+Text Label 8550 6400 0    50   ~ 0
+D23
+Wire Wire Line
+	8200 5250 8200 6300
+Wire Wire Line
+	11750 3950 11750 7700
+Wire Wire Line
+	8200 3950 8200 4900
+Wire Wire Line
+	14700 10050 15800 10050
 $EndSCHEMATC
