File: regius.sch (KiCad schematic (older format))
At the start: 124 parts, among them J1 3.3v, J10 A10, J11 A9, J12 A8, J13 A7, J14 A6, J15 A5, J16 A4, J17 A3, J18 A2, J2 D3, J20 D27, J21 D26, J24 D23, J25 D22, J26 D12, J27 D11, J28 D10, J29 D9, J3 D2, J30 D8, J31 D7, J32 D6, J33 D5, J34 D4, J35 D44, J36 D43, J37 D42, J38 D41, J39 D40, J4 A15, J40 CAN, J41 I2C, J42 D37, J43 D36, J44 D35, J45 D34, J46 D33, J47 D32, J48 D31, J49 D30, J5 A14, J50 D29, J57 D52, J58 D50, J59 D49, J6 A13, J60 D48, J61 D47, J62 D46, J63 D45, J64 DAC, J65 AREF, J66 DAC, J67 Conn_02x05_Counter_Clockwise, J68 TXRX1CAN, J69 4WIRELED, J7 VCC, J70 TXRX, J71 Micro_SD_Card_Det, J72 I2C, J73 I2C, J74 USB_B_Micro, J75 I2C, J76 I2C, J77 I2C, J78 I2C, J79 I2C, J8 A12, J80 I2C, J9 A11, SW1 Reset, U1 GD25Q32CTIGR, U2 samd51p20, U3 TCA9548APWR, U5 LM1117-3.3, Y1 Crystal

Commit message: update layout
Connections:
- net usb_rx_+ renamed +
- net usb_tx_- renamed -
Changed lines of the file:
@@
 $EndComp
 Text Label 23000 7650 0    50   ~ 0
-usb_rx_+
++
 Text Label 23000 7750 0    50   ~ 0
-usb_tx_-
+-
 $Comp
 L Connector:USB_B_Micro J74
@@
 $EndComp
 Text Label 23850 6650 2    50   ~ 0
-usb_tx_-
+-
 Text Label 23850 6750 2    50   ~ 0
-usb_rx_+
++
 Wire Wire Line
 	25200 6350 25200 6150

Commit message: update layout
Parts:
- added J19: reset, Connector_PinHeader_2.54mm:PinHeader_1x02_P2.54mm_Vertical, symbol Connector_Generic:Conn_01x02
- added J22: D28, Connector_PinHeader_2.54mm:PinHeader_1x02_P2.54mm_Vertical, symbol Connector_Generic:Conn_01x02
Connections:
- net D28: now also J22.1 (Pin_1)
- net GND: now also J19.2 (Pin_2), J22.2 (Pin_2)
- net RESET: no longer R9.2, U3.3 (~RESET)
- new net: J19.1 (Pin_1), R9.2, U3.3 (~RESET)
Changed lines of the file:
@@
 Text Label 19200 6250 1    50   ~ 0
-RESET
-Text Label 22700 10550 2    50   ~ 0
 RESET
 Wire Wire Line
@@
 Connection ~ 23350 12150
 Wire Wire Line
-	23350 12150 20900 12150
+	23350 12150 22800 12150
 $Comp
 L power:+3.3V #PWR0101
@@
 D23
 Wire Wire Line
-	8200 5250 8200 6300
+	8200 5250 8200 5550
 Wire Wire Line
 	11750 3950 11750 7700
@@
 Wire Wire Line
 	14700 10050 15800 10050
+$Comp
+L Connector_Generic:Conn_01x02 J19
+U 1 1 5CCCBBE8
+P 22500 10550
+F 0 "J19" V 22580 10542 50  0000 L CNN
+F 1 "reset" H 22580 10451 50  0000 L CNN
+F 2 "Connector_PinHeader_2.54mm:PinHeader_1x02_P2.54mm_Vertical" H 22500 10550 50  0001 C CNN
+F 3 "~" H 22500 10550 50  0001 C CNN
+	1    22500 10550
+	-1   0    0    1
+$EndComp
+Wire Wire Line
+	22800 12150 22800 10450
+Wire Wire Line
+	22800 10450 22700 10450
+Connection ~ 22800 12150
+Wire Wire Line
+	22800 12150 20900 12150
+$Comp
+L Connector_Generic:Conn_01x02 J22
+U 1 1 5D4A2E47
+P 7800 5650
+F 0 "J22" H 7880 5642 50  0000 L CNN
+F 1 "D28" V 8100 5400 50  0000 L CNN
+F 2 "Connector_PinHeader_2.54mm:PinHeader_1x02_P2.54mm_Vertical" H 7800 5650 50  0001 C CNN
+F 3 "~" H 7800 5650 50  0001 C CNN
+	1    7800 5650
+	-1   0    0    1
+$EndComp
+Wire Wire Line
+	8000 5550 8200 5550
+Connection ~ 8200 5550
+Wire Wire Line
+	8200 5550 8200 6300
+Wire Wire Line
+	8000 5650 8550 5650
+Text Label 8550 5650 0    50   ~ 0
+D28
 $EndSCHEMATC

Commit message: update layout
Parts:
- removed J57: D52, Connector_PinHeader_2.54mm:PinHeader_1x02_P2.54mm_Vertical, symbol Connector_Generic:Conn_01x02
- removed J58: D50, Connector_PinHeader_2.54mm:PinHeader_1x02_P2.54mm_Vertical, symbol Connector_Generic:Conn_01x02
- removed J69: 4WIRELED, Connector_PinHeader_2.54mm:PinHeader_1x02_P2.54mm_Vertical, symbol Connector_Generic:Conn_01x02
- removed J72: I2C, Connector_PinHeader_2.54mm:PinHeader_1x02_P2.54mm_Vertical, symbol Connector_Generic:Conn_01x02
- added J23: Conn_01x04, Connector_PinHeader_2.54mm:PinHeader_1x04_P2.54mm_Vertical, symbol Connector_Generic:Conn_01x04
Connections:
- net at U2.47 (PD08): now also J23.4 (Pin_4)
- net at U2.48 (PD09): now also J23.3 (Pin_3)
- net at U2.49 (PD10): now also J23.2 (Pin_2)
- net at U2.50 (PD11): now also J23.1 (Pin_1)
Changed lines of the file:
@@
 Wire Wire Line
 	15450 9550 15450 10550
-Wire Wire Line
-	21600 8550 22700 8550
-Wire Wire Line
-	21600 8450 22700 8450
-$Comp
-L Connector_Generic:Conn_01x02 J72
-U 1 1 5D067002
-P 22900 8450
-F 0 "J72" H 22980 8442 50  0000 L CNN
-F 1 "I2C" H 22980 8351 50  0000 L CNN
-F 2 "Connector_PinHeader_2.54mm:PinHeader_1x02_P2.54mm_Vertical" H 22900 8450 50  0001 C CNN
-F 3 "~" H 22900 8450 50  0001 C CNN
-	1    22900 8450
-	1    0    0    -1
-$EndComp
 $Comp
 L Connector_Generic:Conn_01x02 J73
@@
 Text Label 16950 11500 1    50   ~ 0
 D49
-Wire Wire Line
-	19200 11150 19200 12100
-$Comp
-L Connector_Generic:Conn_01x02 J57
-U 1 1 5D383949
-P 11350 7800
-F 0 "J57" H 11430 7792 50  0000 L CNN
-F 1 "D52" V 11650 7550 50  0000 L CNN
-F 2 "Connector_PinHeader_2.54mm:PinHeader_1x02_P2.54mm_Vertical" H 11350 7800 50  0001 C CNN
-F 3 "~" H 11350 7800 50  0001 C CNN
-	1    11350 7800
-	-1   0    0    1
-$EndComp
-Wire Wire Line
-	11550 7700 11750 7700
-Wire Wire Line
-	11550 7800 12100 7800
-Text Label 12100 7800 0    50   ~ 0
-D52
-$Comp
-L Connector_Generic:Conn_01x02 J58
-U 1 1 5D383952
-P 11350 8150
-F 0 "J58" H 11430 8142 50  0000 L CNN
-F 1 "D50" V 11650 7900 50  0000 L CNN
-F 2 "Connector_PinHeader_2.54mm:PinHeader_1x02_P2.54mm_Vertical" H 11350 8150 50  0001 C CNN
-F 3 "~" H 11350 8150 50  0001 C CNN
-	1    11350 8150
-	-1   0    0    1
-$EndComp
-Wire Wire Line
-	11550 8050 11750 8050
-Wire Wire Line
-	11550 8150 12100 8150
-Text Label 12100 8150 0    50   ~ 0
-D50
 $Comp
 L Connector_Generic:Conn_01x02 J59
@@
 A2
 Wire Wire Line
-	19300 11150 19300 12100
-$Comp
-L Connector_Generic:Conn_01x02 J69
-U 1 1 5E9CBC2B
-P 19300 12300
-F 0 "J69" H 19380 12292 50  0000 L CNN
-F 1 "4WIRELED" H 19380 12201 50  0000 L CNN
-F 2 "Connector_PinHeader_2.54mm:PinHeader_1x02_P2.54mm_Vertical" H 19300 12300 50  0001 C CNN
-F 3 "~" H 19300 12300 50  0001 C CNN
-	1    19300 12300
-	0    1    1    0
-$EndComp
-Wire Wire Line
 	11750 9800 11750 9450
-Connection ~ 11750 7700
-Connection ~ 11750 8050
-Wire Wire Line
-	11750 8050 11750 7700
 Connection ~ 11750 8400
-Wire Wire Line
-	11750 8400 11750 8050
 Connection ~ 11750 8750
 Wire Wire Line
@@
 	8200 5250 8200 5550
 Wire Wire Line
-	11750 3950 11750 7700
-Wire Wire Line
 	8200 3950 8200 4900
 Wire Wire Line
@@
 Text Label 8550 5650 0    50   ~ 0
 D28
+Wire Wire Line
+	19500 11150 19500 12800
+Wire Wire Line
+	19400 11150 19400 12800
+Wire Wire Line
+	19300 11150 19300 12800
+Wire Wire Line
+	19200 11150 19200 12800
+$Comp
+L Connector_Generic:Conn_01x04 J23
+U 1 1 5DA67D42
+P 19400 13000
+F 0 "J23" V 19273 13180 50  0000 L CNN
+F 1 "Conn_01x04" V 19364 13180 50  0000 L CNN
+F 2 "Connector_PinHeader_2.54mm:PinHeader_1x04_P2.54mm_Vertical" H 19400 13000 50  0001 C CNN
+F 3 "~" H 19400 13000 50  0001 C CNN
+	1    19400 13000
+	0    1    1    0
+$EndComp
+Wire Wire Line
+	11750 3950 11750 8400
 $EndSCHEMATC
