File: electrosprawl.kicad_pcb (KiCad board)
At the start: 2 copper layers, 71 x 84 mm, 122 parts, among them J1 3.3v, J10 A10, J11 A9, J12 A8, J13 A7, J14 A6, J15 A5, J16 A4, J17 A3, J18 A2, J19 reset, J2 D3, J20 D27, J21 D26, J22 D28, J23 Conn_01x04, J24 D23, J25 D22, J26 D12, J27 D11, J28 D10, J29 D9, J3 D2, J30 D8, J31 D7, J32 D6, J33 D5, J34 D4, J35 D44, J36 D43, J37 D42, J38 D41, J39 D40, J4 A15, J40 CAN, J41 I2C, J42 D37, J43 D36, J44 D35, J45 D34, J46 D33, J47 D32, J48 D31, J49 D30, J5 A14, J50 D29, J59 D49, J6 A13, J60 D48, J61 D47, J62 D46, J63 D45, J64 DAC, J65 AREF, J66 DAC, J67 Conn_02x05_Counter_Clockwise, J68 TXRX1CAN, J7 VCC, J70 TXRX, J71 Micro_SD_Card_Det, J73 I2C, J74 USB_B_Micro, J75 I2C, J76 I2C, J77 I2C, J78 I2C, J79 I2C, J8 A12, J80 I2C, J9 A11, SW1 Reset, U1 GD25Q32CTIGR, U2 samd51p20, U3 TCA9548APWR, U5 LM1117-3.3, Y1 Crystal

Commit message: update layout
Parts:
- removed J19: reset, Connector_PinHeader_2.54mm:PinHeader_1x02_P2.54mm_Vertical
- removed J41, J73, J75, J76, J77, J78, J79, J80: I2C, Connector_PinHeader_2.54mm:PinHeader_1x02_P2.54mm_Vertical
- removed JP1, JP2, JP3: SolderJumper_2_Open, Jumper:SolderJumper-2_P1.3mm_Open_RoundedPad1.0x1.5mm
- removed R10, R11, R12, R9: R10K, Resistor_SMD:R_0603_1608Metric
- removed U3: TCA9548APWR, Package_SO:TSSOP-24_4.4x7.8mm_P0.65mm
- moved J44 25.4 mm to (166.9, 68.9), turned to 90 degrees
- moved J61 12.2 mm to (104.0, 90.9)
- moved J35 12.0 mm to (118.5, 98.9)
- moved J39 10.7 mm to (123.7, 98.9)
- moved H3 10.2 mm to (99.5, 109.9)
- moved J37 8.50 mm to (130.0, 98.9)
- moved R7 7.64 mm to (154.1, 71.7)
- moved J21 6.73 mm to (136.5, 99.2)
- moved J43 5.89 mm to (146.7, 99.1)
- moved J45 5.59 mm to (151.2, 99.1)
- moved J24 5.49 mm to (141.7, 99.1)
- moved J59 5.17 mm to (113.0, 98.7)
- moved J25 5.16 mm to (121.5, 90.8)
- moved J62 3.91 mm to (109.7, 90.8)
- moved R8 3.76 mm to (157.5, 71.7)
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Routing:
- net Net-(J75-Pad2): track 42.1 -> 0.00 mm, vias 1 -> 0
- net Net-(J75-Pad1): track 32.0 -> 0.00 mm, vias 1 -> 0
- net Net-(J19-Pad1): track 30.6 -> 0.00 mm
- net /D35: track 32.3 -> 5.62 mm, vias 1 -> 0
- net Net-(J76-Pad2): track 21.9 -> 0.00 mm
- net Net-(J76-Pad1): track 19.4 -> 0.00 mm, vias 1 -> 0
- net Net-(J80-Pad2): track 17.9 -> 0.00 mm
- net Net-(J41-Pad2): track 17.2 -> 0.00 mm, vias 1 -> 0
- net Net-(R7-Pad2): track 27.7 -> 10.6 mm
- net Net-(J73-Pad2): track 17.0 -> 0.00 mm, vias 1 -> 0
- net Net-(J73-Pad1): track 16.7 -> 0.00 mm, vias 1 -> 0
- net Net-(R8-Pad2): track 31.2 -> 15.2 mm, vias 2 -> 0
- net Net-(J79-Pad2): track 15.9 -> 0.00 mm
- net Net-(J78-Pad2): track 15.7 -> 0.00 mm
- net Net-(J80-Pad1): track 15.4 -> 0.00 mm
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- removed copper zone on B.Cu, net +3V3
Other:
- board size 71 x 84 mm -> 74 x 90.3 mm

Commit message: update layout redesign
Parts:
- removed J40: CAN, Connector_PinHeader_2.54mm:PinHeader_1x03_P2.54mm_Vertical
- removed J68: TXRX1CAN, Connector_PinHeader_2.54mm:PinHeader_1x03_P2.54mm_Vertical
- removed U1: GD25Q32CTIGR, GD25Q32CTIGR:SOIC127P600X175-8N
- moved J25 21.9 mm to (123.6, 112.6)
- moved J16 21.5 mm to (104.3, 45.0), turned to 0 degrees
- moved J66 17.8 mm to (104.3, 77.1), turned to 0 degrees
- moved J12 17.4 mm to (104.3, 61.1), turned to 0 degrees
- moved J14 14.7 mm to (110.1, 53.1), turned to 0 degrees
- moved J64 14.2 mm to (104.3, 53.1), turned to 0 degrees
- moved J17 13.1 mm to (110.1, 45.0), turned to 0 degrees
- moved J60 12.8 mm to (104.3, 85.1)
- moved J23 12.5 mm to (132.6, 76.0), turned to 270 degrees
- moved J65 12.4 mm to (115.6, 61.1), turned to 0 degrees
- moved J18 11.2 mm to (115.6, 45.0), turned to 0 degrees
- moved J9 10.8 mm to (104.3, 69.1), turned to 0 degrees
- moved J10 10.7 mm to (110.1, 69.1), turned to 0 degrees
- moved J15 8.99 mm to (115.6, 53.1), turned to 0 degrees
- moved J5 6.56 mm to (115.6, 85.1), turned to 0 degrees
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Routing:
- net /D22: track 32.2 -> 8.79 mm, vias 1 -> 0
- net /A4: track 10.0 -> 32.2 mm
- net Net-(J23-Pad4): track 22.9 -> 1.40 mm
- net Net-(U1-Pad7): track 18.4 -> 0.00 mm, vias 2 -> 0
- net Net-(J23-Pad3): track 18.1 -> 1.75 mm
- net Net-(U1-Pad6): track 15.9 -> 0.00 mm
- net /D48: track 29.9 -> 45.6 mm, vias 2 -> 0
- net /A8: track 13.2 -> 28.8 mm, vias 1 -> 0
- net Net-(J66-Pad1): track 25.4 -> 40.1 mm, vias 1 -> 0
- net Net-(U1-Pad5): track 12.9 -> 0.00 mm, vias 2 -> 0
- net /A10: track 15.3 -> 28.1 mm
- net /D46: track 32.9 -> 45.5 mm, vias 1 -> 0
- net /D47: track 39.3 -> 51.4 mm, vias 1 -> 0
- net Net-(J23-Pad2): track 15.2 -> 3.56 mm
- net Net-(J65-Pad1): track 26.0 -> 14.7 mm, vias 1 -> 0
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
Commit message: update layout redesign
Parts:
- moved J25 27.9 mm to (125.0, 84.7)
- moved J1 27.4 mm to (167.9, 74.1)
- moved J45 25.3 mm to (162.2, 76.3)
- moved J43 19.2 mm to (158.2, 83.8)
- moved J70 16.6 mm to (170.7, 34.1), turned to 0 degrees
- moved J37 15.1 mm to (135.5, 84.8)
- moved J42 14.8 mm to (154.7, 76.0)
- moved J36 11.8 mm to (130.2, 100.8)
- moved J20 11.5 mm to (135.5, 100.8)
- moved J39 8.91 mm to (130.2, 92.8)
- moved J22 7.84 mm to (140.7, 84.8)
- moved J35 6.43 mm to (125.0, 100.8)
- moved J21 6.41 mm to (135.5, 92.8)
- moved J24 6.37 mm to (140.7, 92.8)
- moved J38 6.29 mm to (130.2, 84.8)
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Routing:
- net /D34: track 33.9 -> 0.00 mm
- net /D36: track 32.9 -> 0.00 mm
- net /D37: track 25.9 -> 0.00 mm, vias 1 -> 0
- net Net-(J23-Pad4): track 1.40 -> 17.5 mm, vias 1 -> 0
- net /D42: track 33.7 -> 17.7 mm, vias 1 -> 0
- net /D43: track 22.5 -> 36.4 mm
- net Net-(J68-Pad1): track 13.9 -> 0.00 mm
- net /D22: track 8.79 -> 22.5 mm
- net Net-(J23-Pad3): track 1.75 -> 15.4 mm, vias 1 -> 0
- net /D10: track 22.8 -> 10.1 mm
- net /D27: track 21.2 -> 33.5 mm
- net Net-(J68-Pad2): track 11.2 -> 0.00 mm
- net /D39: track 11.1 -> 0.00 mm
- net Net-(J70-Pad1): track 21.6 -> 32.2 mm
- net Net-(J70-Pad2): track 23.3 -> 33.3 mm
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
Commit message: update layout
Parts:
- removed J1: 3.3v, Connector_PinHeader_2.54mm:PinHeader_1x02_P2.54mm_Vertical
- added J40: Conn_01x02, Connector_PinHeader_2.54mm:PinHeader_1x02_P2.54mm_Vertical, F.Cu at (131.4, 75.8)
- added J53: Conn_01x02, Connector_PinHeader_2.54mm:PinHeader_1x02_P2.54mm_Vertical, F.Cu at (148.6, 79.6)
- added J54: Conn_01x02, Connector_PinHeader_2.54mm:PinHeader_1x02_P2.54mm_Vertical, F.Cu at (148.6, 87.6)
- added J55: Conn_01x02, Connector_PinHeader_2.54mm:PinHeader_1x02_P2.54mm_Vertical, F.Cu at (148.6, 95.6)
- added J56: Conn_01x02, Connector_PinHeader_2.54mm:PinHeader_1x02_P2.54mm_Vertical, F.Cu at (140.7, 100.9)
- added J57: Conn_01x02, Connector_PinHeader_2.54mm:PinHeader_1x02_P2.54mm_Vertical, F.Cu at (148.6, 103.6)
- added J58: Conn_01x02, Connector_PinHeader_2.54mm:PinHeader_1x02_P2.54mm_Vertical, F.Cu at (154.1, 103.6)
- added J69: Conn_01x02, Connector_PinHeader_2.54mm:PinHeader_1x02_P2.54mm_Vertical, F.Cu at (159.6, 103.6)
- added J72: Conn_01x02, Connector_PinHeader_2.54mm:PinHeader_1x02_P2.54mm_Vertical, F.Cu at (165.1, 103.6)
- added J84: Conn_01x02, Connector_PinHeader_2.54mm:PinHeader_1x02_P2.54mm_Vertical, F.Cu at (154.1, 95.6)
- added J85: Conn_01x02, Connector_PinHeader_2.54mm:PinHeader_1x02_P2.54mm_Vertical, F.Cu at (159.6, 95.6)
- added J86: Conn_01x02, Connector_PinHeader_2.54mm:PinHeader_1x02_P2.54mm_Vertical, F.Cu at (165.1, 95.6)
- added J87: Conn_01x02, Connector_PinHeader_2.54mm:PinHeader_1x02_P2.54mm_Vertical, F.Cu at (170.6, 95.6)
- added J88: Conn_01x02, Connector_PinHeader_2.54mm:PinHeader_1x02_P2.54mm_Vertical, F.Cu at (165.1, 87.6)
- added J89: Conn_01x02, Connector_PinHeader_2.54mm:PinHeader_1x02_P2.54mm_Vertical, F.Cu at (170.6, 87.6)
- added R10: R10K, Resistor_SMD:R_0603_1608Metric, F.Cu at (161.6, 85.6)
- added U3: SX1509, Package_DFN_QFN:QFN-28-1EP_4x4mm_P0.45mm_EP2.4x2.4mm, F.Cu at (156.6, 89.9)
- J32: value D6 -> Conn_01x02
- moved J32 28.6 mm to (124.3, 72.6), turned to 0 degrees
- moved J46 18.9 mm to (170.6, 55.5), turned to 0 degrees
- moved J47 14.2 mm to (165.1, 55.5), turned to 0 degrees
- moved R7 13.9 mm to (153.1, 85.6), turned to 0 degrees
- moved R8 13.9 mm to (156.7, 85.6), turned to 0 degrees
- moved J31 13.1 mm to (154.1, 63.5), turned to 0 degrees
- moved J33 13.0 mm to (170.6, 71.6), turned to 0 degrees
- moved J50 12.8 mm to (165.1, 63.5), turned to 0 degrees
- moved J44 10.8 mm to (165.1, 79.6), turned to 0 degrees
- moved J45 8.99 mm to (170.6, 79.6)
- moved J2 8.10 mm to (159.6, 71.6), turned to 0 degrees
- moved J34 6.91 mm to (165.1, 71.6), turned to 0 degrees
- moved H3 6.45 mm to (104.2, 105.5)
- moved J3 5.98 mm to (154.1, 71.6), turned to 0 degrees
- moved J43 4.42 mm to (159.6, 79.6)
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Connections:
- net /D38 renamed Net-(U2-Pad44)
- net /D39 renamed Net-(U2-Pad43)
- J32 pad 1: /D6 -> Net-(J32-Pad1)
- R8 pad 1: +3V3 -> Net-(R8-Pad1)
- R8 pad 2: Net-(R8-Pad2) -> +3V3
- U2 pad 33: Net-(U1-Pad5) -> Net-(J32-Pad1)
- U2 pad 37: +3V3 -> Net-(U2-Pad37)
- U2 pad 38: GND -> Net-(U2-Pad38)
- U2 pad 71: Net-(R8-Pad2) -> Net-(R8-Pad1)
- U2 pad 80: /D6 -> Net-(U2-Pad80)
Routing:
- net /D34: track 0.00 -> 31.9 mm
- net Net-(R8-Pad1): track 0.00 -> 30.9 mm, vias 0 -> 2
- net /+: track 25.8 -> 0.00 mm
- net /-: track 25.8 -> 0.00 mm
- net Net-(J72-Pad1): track 0.00 -> 24.8 mm
- net Net-(J56-Pad1): track 0.00 -> 23.1 mm
- net /D35: track 5.62 -> 26.1 mm
- net /D36: track 0.00 -> 20.4 mm
- net Net-(J69-Pad1): track 0.00 -> 20.0 mm
- net Net-(R7-Pad2): track 10.6 -> 29.0 mm, vias 0 -> 2
- net Net-(J58-Pad1): track 0.00 -> 16.7 mm
- net Net-(J57-Pad1): track 0.00 -> 16.4 mm
- net /D37: track 0.00 -> 15.6 mm
- net /D10: track 10.1 -> 25.6 mm
- net Net-(R8-Pad2): track 15.2 -> 0.00 mm
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Other:
- board size 74 x 90.3 mm -> 73.8 x 86.2 mm

Commit message: update layout
Parts:
- added J1: 3.3v, Connector_PinHeader_2.54mm:PinHeader_1x02_P2.54mm_Vertical, F.Cu at (115.6, 100.8)
- added J68: Conn_01x02, Connector_PinHeader_2.54mm:PinHeader_1x02_P2.54mm_Vertical, F.Cu at (170.6, 63.6)
- moved C10 4.16 mm to (119.6, 34.1), turned to 0 degrees
- moved D6 4.16 mm to (107.1, 38.5)
- moved R13 4.16 mm to (111.5, 38.5)
- moved J7 2.78 mm to (114.3, 26.1)
- moved C9 2.21 mm to (121.2, 28.6)
- moved U5 1.98 mm to (111.3, 33.3)
- moved R8 1.21 mm to (157.8, 85.3)
- moved R10 0.88 mm to (161.1, 86.3)
- moved C15 0.55 mm to (139.1, 50.8)
- moved R2 0.34 mm to (132.1, 37.4)
- moved C5 0.19 mm to (123.9, 59.0)
- moved C19 0.11 mm to (150.2, 58.0)
Connections:
- J53 pad 2: GND -> Net-(J53-Pad2)
- J54 pad 2: GND -> Net-(J53-Pad2)
- J55 pad 2: GND -> Net-(J53-Pad2)
- J56 pad 2: GND -> Net-(J53-Pad2)
- J57 pad 2: GND -> Net-(J53-Pad2)
- J58 pad 2: GND -> Net-(J53-Pad2)
- J69 pad 2: GND -> Net-(J53-Pad2)
- J72 pad 2: GND -> Net-(J53-Pad2)
- J84 pad 2: GND -> Net-(J53-Pad2)
- J85 pad 2: GND -> Net-(J53-Pad2)
- J86 pad 2: GND -> Net-(J53-Pad2)
- J87 pad 2: GND -> Net-(J53-Pad2)
- J88 pad 2: GND -> Net-(J53-Pad2)
- J89 pad 2: GND -> Net-(J53-Pad2)
- U2 pad 37: Net-(U2-Pad37) -> +3V3
- U2 pad 38: Net-(U2-Pad38) -> GND
Routing:
- net /-: track 0.00 -> 28.5 mm
- net /+: track 0.00 -> 28.5 mm
- net Net-(J68-Pad2): track 0.00 -> 28.2 mm
- net Net-(J68-Pad1): track 0.00 -> 27.3 mm
- net VCC: track 0.00 -> 13.8 mm
- net Net-(J67-Pad9): track 10.8 -> 22.5 mm
- net +3V3: track 60.8 -> 70.8 mm, vias 16 -> 20
- net /SDCD: track 60.3 -> 63.2 mm, vias 3 -> 2
- net /D30: track 8.71 -> 10.5 mm
- net Net-(R4-Pad1): track 21.1 -> 22.5 mm
- net /D5: track 28.7 -> 30.1 mm
- net Net-(R5-Pad1): track 22.6 -> 23.6 mm
- net /D34: track 31.9 -> 32.9 mm
- net Net-(R10-Pad1): track 4.69 -> 3.89 mm
- net Net-(D4-Pad4): track 27.5 -> 28.1 mm
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- added copper zone on B.Cu, net +3V3
Other:
- net class vcc added: clearance 0.1, trace_width 1.5, via_dia 0.45, via_drill 0.35

Commit message: update redesign
Parts:
- removed J10: A10, Connector_PinHeader_2.54mm:PinHeader_1x02_P2.54mm_Vertical
- removed J11: A9, Connector_PinHeader_2.54mm:PinHeader_1x02_P2.54mm_Vertical
- removed J12: A8, Connector_PinHeader_2.54mm:PinHeader_1x02_P2.54mm_Vertical
- removed J13: A7, Connector_PinHeader_2.54mm:PinHeader_1x02_P2.54mm_Vertical
- removed J14: A6, Connector_PinHeader_2.54mm:PinHeader_1x02_P2.54mm_Vertical
- removed J15: A5, Connector_PinHeader_2.54mm:PinHeader_1x02_P2.54mm_Vertical
- removed J16: A4, Connector_PinHeader_2.54mm:PinHeader_1x02_P2.54mm_Vertical
- removed J17: A3, Connector_PinHeader_2.54mm:PinHeader_1x02_P2.54mm_Vertical
- removed J18: A2, Connector_PinHeader_2.54mm:PinHeader_1x02_P2.54mm_Vertical
- removed J20: D27, Connector_PinHeader_2.54mm:PinHeader_1x02_P2.54mm_Vertical
- removed J21: D26, Connector_PinHeader_2.54mm:PinHeader_1x02_P2.54mm_Vertical
- removed J22: D28, Connector_PinHeader_2.54mm:PinHeader_1x02_P2.54mm_Vertical
- removed J24: D23, Connector_PinHeader_2.54mm:PinHeader_1x02_P2.54mm_Vertical
- removed J25: D22, Connector_PinHeader_2.54mm:PinHeader_1x02_P2.54mm_Vertical
- removed J3: D2, Connector_PinHeader_2.54mm:PinHeader_1x02_P2.54mm_Vertical
- removed J30: D8, Connector_PinHeader_2.54mm:PinHeader_1x02_P2.54mm_Vertical
- removed J31: D7, Connector_PinHeader_2.54mm:PinHeader_1x02_P2.54mm_Vertical
- removed J32: Conn_01x02, Connector_PinHeader_2.54mm:PinHeader_1x02_P2.54mm_Vertical
- removed J33: D5, Connector_PinHeader_2.54mm:PinHeader_1x02_P2.54mm_Vertical
- removed J34: D4, Connector_PinHeader_2.54mm:PinHeader_1x02_P2.54mm_Vertical
- removed J35: D44, Connector_PinHeader_2.54mm:PinHeader_1x02_P2.54mm_Vertical
- removed J36: D43, Connector_PinHeader_2.54mm:PinHeader_1x02_P2.54mm_Vertical
- removed J37: D42, Connector_PinHeader_2.54mm:PinHeader_1x02_P2.54mm_Vertical
- removed J38: D41, Connector_PinHeader_2.54mm:PinHeader_1x02_P2.54mm_Vertical
- removed J39: D40, Connector_PinHeader_2.54mm:PinHeader_1x02_P2.54mm_Vertical
- removed J4: A15, Connector_PinHeader_2.54mm:PinHeader_1x02_P2.54mm_Vertical
- removed J42: D37, Connector_PinHeader_2.54mm:PinHeader_1x02_P2.54mm_Vertical
- removed J43: D36, Connector_PinHeader_2.54mm:PinHeader_1x02_P2.54mm_Vertical
- removed J44: D35, Connector_PinHeader_2.54mm:PinHeader_1x02_P2.54mm_Vertical
- removed J45: D34, Connector_PinHeader_2.54mm:PinHeader_1x02_P2.54mm_Vertical
- removed J46: D33, Connector_PinHeader_2.54mm:PinHeader_1x02_P2.54mm_Vertical
- removed J47: D32, Connector_PinHeader_2.54mm:PinHeader_1x02_P2.54mm_Vertical
- removed J48: D31, Connector_PinHeader_2.54mm:PinHeader_1x02_P2.54mm_Vertical
- removed J49: D30, Connector_PinHeader_2.54mm:PinHeader_1x02_P2.54mm_Vertical
- removed J5: A14, Connector_PinHeader_2.54mm:PinHeader_1x02_P2.54mm_Vertical
- removed J50: D29, Connector_PinHeader_2.54mm:PinHeader_1x02_P2.54mm_Vertical
- removed J59: D49, Connector_PinHeader_2.54mm:PinHeader_1x02_P2.54mm_Vertical
- removed J6: A13, Connector_PinHeader_2.54mm:PinHeader_1x02_P2.54mm_Vertical
- removed J60: D48, Connector_PinHeader_2.54mm:PinHeader_1x02_P2.54mm_Vertical
- removed J61: D47, Connector_PinHeader_2.54mm:PinHeader_1x02_P2.54mm_Vertical
- removed J62: D46, Connector_PinHeader_2.54mm:PinHeader_1x02_P2.54mm_Vertical
- removed J63: D45, Connector_PinHeader_2.54mm:PinHeader_1x02_P2.54mm_Vertical
- removed J64, J66: DAC, Connector_PinHeader_2.54mm:PinHeader_1x02_P2.54mm_Vertical
- removed J65: AREF, Connector_PinHeader_2.54mm:PinHeader_1x02_P2.54mm_Vertical
- removed J8: A12, Connector_PinHeader_2.54mm:PinHeader_1x02_P2.54mm_Vertical
- removed J9: A11, Connector_PinHeader_2.54mm:PinHeader_1x02_P2.54mm_Vertical
- J2: value D3 -> Conn_02x08_Odd_Even
Connections:
- J2 pad 1: /D3 -> Net-(J2-Pad1)
- J2 pad 2: GND -> /A2
- J26 pad 2: GND -> Net-(J26-Pad2)
- J27 pad 2: GND -> Net-(J26-Pad2)
- J28 pad 2: GND -> Net-(J26-Pad2)
- J29 pad 2: GND -> Net-(J26-Pad2)
Routing:
- net /D47: track 51.4 -> 6.81 mm
- net /D46: track 45.5 -> 6.91 mm
- net /D48: track 45.6 -> 7.24 mm
- net /A15: track 40.4 -> 7.63 mm
- net Net-(J66-Pad1): track 40.1 -> 8.03 mm
- net /D49: track 34.6 -> 7.01 mm
- net /A13: track 34.4 -> 8.23 mm
- net /A11: track 34.2 -> 8.63 mm
- net /A4: track 32.2 -> 6.66 mm
- net /A14: track 30.1 -> 7.83 mm
- net /A8: track 28.8 -> 8.11 mm
- net /A3: track 26.4 -> 6.30 mm
- net Net-(J64-Pad1): track 28.2 -> 8.65 mm
- net /A10: track 28.1 -> 8.83 mm
- net /A12: track 23.4 -> 8.43 mm
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- removed copper zone on B.Cu, net +3V3

Commit message: update redesign
Parts:
- removed D4, D5: WS2812B, LED_SMD:LED_WS2812B_PLCC4_5.0x5.0mm_P3.2mm
- removed J1: 3.3v, Connector_PinHeader_2.54mm:PinHeader_1x02_P2.54mm_Vertical
- removed J2: Conn_02x08_Odd_Even, Connector_PinHeader_2.54mm:PinHeader_1x02_P2.54mm_Vertical
- removed J23: Conn_01x04, Connector_PinHeader_2.54mm:PinHeader_1x04_P2.54mm_Vertical
- removed J27: D11, Connector_PinHeader_2.54mm:PinHeader_1x02_P2.54mm_Vertical
- removed J28: D10, Connector_PinHeader_2.54mm:PinHeader_1x02_P2.54mm_Vertical
- removed J40, J53, J54, J55, J56, J57, J58, J68, J69, J72, J84, J85, J86, J87, J88, J89: Conn_01x02, Connector_PinHeader_2.54mm:PinHeader_1x02_P2.54mm_Vertical
- removed J70: TXRX, Connector_PinHeader_2.54mm:PinHeader_1x03_P2.54mm_Vertical
- removed R10, R7, R8: R10K, Resistor_SMD:R_0603_1608Metric
- removed U3: SX1509, Package_DFN_QFN:QFN-28-1EP_4x4mm_P0.45mm_EP2.4x2.4mm
- moved D6 51.2 mm to (158.3, 36.8), turned to 270 degrees
- moved R13 47.2 mm to (158.3, 32.5), turned to 90 degrees
- moved J26 16.8 mm to (111.7, 37.5)
- moved J7 12.9 mm to (127.3, 25.7), turned to 90 degrees
- moved J74 11.3 mm to (160.7, 52.4)
- moved H5 11.0 mm to (159.5, 26.7)
- moved U5 10.0 mm to (120.5, 29.1), turned to 90 degrees
- moved J71 9.85 mm to (148.5, 30.4)
- moved SW1 9.69 mm to (137.5, 30.6), turned to 90 degrees
- moved J29 9.50 mm to (111.7, 45.3)
- moved C9 9.45 mm to (122.8, 37.9), turned to 270 degrees
- moved H4 7.76 mm to (112.0, 26.5)
- moved C10 4.47 mm to (117.3, 37.9), turned to 270 degrees
- moved C19 2.37 mm to (148.0, 58.9)
- moved C18 2.30 mm to (139.4, 73.4)
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Routing:
- net /SDCD: track 63.2 -> 2.58 mm, vias 2 -> 0
- net /D44: track 40.4 -> 0.00 mm
- net Net-(J70-Pad1): track 39.7 -> 0.00 mm, vias 1 -> 0
- net Net-(J70-Pad2): track 37.3 -> 0.00 mm, vias 1 -> 0
- net /D43: track 36.4 -> 0.00 mm
- net /D27: track 33.5 -> 0.00 mm
- net /D34: track 32.9 -> 0.00 mm
- net Net-(R8-Pad1): track 31.3 -> 0.00 mm, vias 2 -> 0
- net Net-(J71-Pad3): track 30.8 -> 0.00 mm, vias 2 -> 0
- net /D5: track 30.1 -> 0.00 mm
- net Net-(R7-Pad2): track 29.3 -> 0.00 mm, vias 2 -> 0
- net /D45: track 31.1 -> 2.60 mm
- net /-: track 28.5 -> 0.00 mm
- net /+: track 28.5 -> 0.00 mm
- net Net-(J68-Pad2): track 28.2 -> 0.00 mm
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Other:
- net class vcc: trace_width 1.5 -> 1
