File: electrosprawl.kicad_pcb (KiCad board)
At the start: 2 copper layers, 73.8 x 86.2 mm, 45 parts, among them J26 D12, J29 D9, J67 Conn_02x05_Counter_Clockwise, J7 VCC, J71 Micro_SD_Card_Det, J74 USB_B_Micro, SW1 Reset, U2 samd51p20, U5 LM1117-3.3, Y1 Crystal

Commit message: update layout
Parts:
- added J1: 3.3v, Connector_PinHeader_2.54mm:PinHeader_1x02_P2.54mm_Vertical, F.Cu at (199.7, 283.8)
- added J2: Conn_02x08_Counter_Clockwise, Connector_PinHeader_2.54mm:PinHeader_2x08_P2.54mm_Vertical, F.Cu at (118.2, 70.5)
- added J3: Conn_02x04_Counter_Clockwise, Connector_PinHeader_2.54mm:PinHeader_2x04_P2.54mm_Vertical, F.Cu at (126.4, 78.1)
- added J4: Conn_02x04_Counter_Clockwise, Connector_PinHeader_2.54mm:PinHeader_2x04_P2.54mm_Vertical, F.Cu at (147.2, 78.1)
- added J5: Conn_02x08_Counter_Clockwise, Connector_PinHeader_2.54mm:PinHeader_2x08_P2.54mm_Vertical, F.Cu at (152.7, 55.3)
- added J70: TXRX, Connector_PinHeader_2.54mm:PinHeader_1x03_P2.54mm_Vertical, F.Cu at (214.1, 271.5)
- moved J26 17.7 mm to (94.3, 34.5)
- moved J29 14.8 mm to (97.2, 42.5)
- moved J74 6.02 mm to (156.0, 48.5)
- moved C19 0.97 mm to (148.7, 58.3)
- moved C20 0.67 mm to (148.0, 63.0)
- moved C18 0.40 mm to (139.0, 73.4)
Connections:
- net /D22 renamed Net-(U2-Pad51)
- net /D44 renamed Net-(U2-Pad55)
- net /D45 renamed Net-(U2-Pad52)
- net /D7 renamed Net-(U2-Pad81)
- U2 pad 11: /A7 -> Net-(J2-Pad10)
- U2 pad 12: /A8 -> Net-(J2-Pad9)
- U2 pad 128: /A2 -> Net-(J2-Pad16)
- U2 pad 17: /A9 -> Net-(J2-Pad8)
- U2 pad 18: /A10 -> Net-(J2-Pad7)
- U2 pad 19: /A11 -> Net-(J2-Pad6)
- U2 pad 20: /A12 -> Net-(J2-Pad5)
- U2 pad 21: /A13 -> Net-(J2-Pad4)
- U2 pad 23: /A14 -> Net-(J2-Pad2)
- U2 pad 24: /A15 -> Net-(J2-Pad1)
- U2 pad 27: /D48 -> Net-(J3-Pad2)
- U2 pad 28: /D49 -> Net-(J3-Pad1)
- U2 pad 29: /D46 -> Net-(J3-Pad4)
- U2 pad 3: /A3 -> Net-(J2-Pad15)
- U2 pad 30: /D47 -> Net-(J3-Pad3)
- U2 pad 4: /A4 -> Net-(J2-Pad14)
- U2 pad 56: /D41 -> Net-(J4-Pad8)
- U2 pad 57: /D40 -> Net-(J4-Pad7)
- U2 pad 58: /D43 -> Net-(J4-Pad6)
- U2 pad 59: /D42 -> Net-(J4-Pad5)
- U2 pad 60: /D26 -> Net-(J4-Pad4)
- U2 pad 61: /D27 -> Net-(J4-Pad3)
- U2 pad 62: /D28 -> Net-(J4-Pad2)
- U2 pad 63: /D23 -> Net-(J4-Pad1)
- U2 pad 66: /D37 -> Net-(J5-Pad16)
- U2 pad 67: /D36 -> Net-(J5-Pad15)
- U2 pad 68: /D35 -> Net-(J5-Pad14)
- U2 pad 69: /D34 -> Net-(J5-Pad13)
- U2 pad 7: /A5 -> Net-(J2-Pad13)
- U2 pad 72: /D2 -> Net-(J5-Pad12)
- U2 pad 73: /D3 -> Net-(J5-Pad11)
- U2 pad 74: /D4 -> Net-(J5-Pad10)
- U2 pad 75: /D5 -> Net-(J5-Pad9)
- U2 pad 8: /A6 -> Net-(J2-Pad12)
- U2 pad 84: /D8 -> Net-(J5-Pad8)
- U2 pad 85: /D29 -> Net-(J5-Pad7)
- U2 pad 88: /D33 -> Net-(J5-Pad4)
- U2 pad 89: /D32 -> Net-(J5-Pad3)
- U2 pad 92: /D31 -> Net-(J5-Pad2)
- U2 pad 93: /D30 -> Net-(J5-Pad1)
Routing:
- net Net-(J5-Pad16): track 0.00 -> 13.5 mm
- net Net-(J5-Pad14): track 0.00 -> 12.8 mm
- net Net-(J5-Pad12): track 0.00 -> 12.4 mm
- net Net-(J5-Pad8): track 0.00 -> 12.2 mm
- net Net-(J4-Pad2): track 0.00 -> 12.1 mm
- net Net-(J5-Pad2): track 0.00 -> 12.0 mm
- net Net-(J2-Pad16): track 0.00 -> 11.8 mm
- net /A2: track 11.8 -> 0.00 mm
- net Net-(J5-Pad10): track 0.00 -> 11.7 mm
- net Net-(J5-Pad4): track 0.00 -> 11.6 mm
- net Net-(J5-Pad6): track 0.00 -> 11.6 mm
- net Net-(J4-Pad4): track 0.00 -> 11.3 mm
- net Net-(J4-Pad6): track 0.00 -> 10.6 mm
- net Net-(J5-Pad15): track 0.00 -> 10.1 mm
- net Net-(J5-Pad13): track 0.00 -> 9.37 mm
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
Commit message: update redesign
Parts:
- removed D1: LED_Small, LED_SMD:LED_0603_1608Metric
- removed J26: D12, Connector_PinHeader_2.54mm:PinHeader_1x02_P2.54mm_Vertical
- removed J29: D9, Connector_PinHeader_2.54mm:PinHeader_1x02_P2.54mm_Vertical
- removed R3: R1K, Resistor_SMD:R_0603_1608Metric
- J3: value Conn_02x04_Counter_Clockwise -> Conn_02x06_Counter_Clockwise; footprint Connector_PinHeader_2.54mm:PinHeader_2x04_P2.54mm_Vertical -> Connector_PinHeader_2.54mm:PinHeader_2x06_P2.54mm_Vertical
- moved C11 2.59 mm to (131.4, 75.6)
- moved J3 1.95 mm to (128.4, 78.1), turned to 270 degrees
- moved C18 0.85 mm to (138.9, 74.2)
- moved C16 0.84 mm to (136.1, 74.2)
- moved C15 0.25 mm to (138.9, 50.8)
- moved C5 0.20 mm to (123.9, 58.8)
Connections:
- J3 pad 1: Net-(J3-Pad1) -> GND
- J3 pad 2: Net-(J3-Pad2) -> GND
- U2 pad 27: Net-(J3-Pad2) -> Net-(J3-Pad11)
- U2 pad 28: Net-(J3-Pad1) -> Net-(J3-Pad12)
- U2 pad 29: Net-(J3-Pad4) -> Net-(J3-Pad9)
- U2 pad 30: Net-(J3-Pad3) -> Net-(J3-Pad10)
- U2 pad 33: Net-(J3-Pad8) -> Net-(J3-Pad7)
- U2 pad 34: Net-(J3-Pad7) -> Net-(J3-Pad8)
- U2 pad 35: Net-(J3-Pad6) -> Net-(J3-Pad5)
- U2 pad 36: Net-(J3-Pad5) -> Net-(J3-Pad6)
- U2 pad 39: Net-(U2-Pad39) -> Net-(J3-Pad3)
- U2 pad 40: Net-(U2-Pad40) -> Net-(J3-Pad4)
Routing:
- net Net-(J71-Pad8): track 0.00 -> 21.2 mm
- net Net-(J71-Pad7): track 0.00 -> 21.2 mm
- net Net-(J3-Pad12): track 0.00 -> 20.3 mm
- net Net-(J3-Pad11): track 0.00 -> 18.4 mm
- net Net-(J3-Pad10): track 0.00 -> 18.0 mm
- net Net-(R3-Pad1): track 21.9 -> 4.39 mm, vias 2 -> 0
- net Net-(J3-Pad8): track 0.00 -> 16.5 mm
- net Net-(J3-Pad9): track 0.00 -> 16.1 mm
- net Net-(J3-Pad6): track 0.00 -> 14.7 mm
- net Net-(J3-Pad7): track 0.00 -> 14.6 mm
- net Net-(J3-Pad5): track 0.00 -> 11.9 mm
- net Net-(J71-Pad3): track 0.00 -> 11.4 mm, vias 0 -> 2
- net Net-(J3-Pad4): track 6.91 -> 17.8 mm, vias 0 -> 1
- net +3V3: track 57.8 -> 67.8 mm, vias 16 -> 19
- net Net-(R1-Pad1): track 0.00 -> 9.87 mm
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
Commit message: add rgb led
Parts:
- added D1: LED_ARGB, LED_SMD:LED_RGB_5050-6, F.Cu at (114.5, 45.5)
- added J6: 3.3v, Connector_PinHeader_2.54mm:PinHeader_1x02_P2.54mm_Vertical, F.Cu at (126.5, 45.5)
- added R3: R330, Resistor_SMD:R_0603_1608Metric, F.Cu at (121.0, 47.5)
- moved J70 244.6 mm to (159.5, 33.1)
- moved J1 207.9 mm to (155.3, 80.7), turned to 90 degrees
- moved D6 46.5 mm to (111.8, 38.1)
- moved R13 46.5 mm to (111.8, 33.7)
- moved J74 5.30 mm to (160.3, 45.4)
- moved C8 4.71 mm to (140.1, 37.8), turned to 90 degrees
- moved C14 2.50 mm to (144.3, 51.9)
- moved C7 2.11 mm to (136.6, 45.8)
- moved C6 1.21 mm to (136.6, 50.0)
- moved R2 1.13 mm to (131.9, 38.5), turned to 0 degrees
- moved C13 0.81 mm to (134.7, 50.0)
- moved C19 0.75 mm to (149.5, 58.2)
Connections:
- net /RESET renamed Net-(C8-Pad1)
- U2 pad 126: Net-(R3-Pad1) -> /D13
Routing:
- net /SDCD: track 2.58 -> 54.6 mm, vias 0 -> 2
- net /D9: track 3.02 -> 25.6 mm
- net /+: track 0.00 -> 22.2 mm
- net /-: track 0.00 -> 22.2 mm
- net /D13: track 0.00 -> 13.5 mm
- net Net-(J71-Pad5): track 9.84 -> 23.2 mm
- net /D12: track 7.30 -> 20.4 mm
- net Net-(J71-Pad3): track 11.4 -> 24.3 mm
- net Net-(J6-Pad1): track 10.2 -> 18.9 mm, vias 0 -> 1
- net Net-(R3-Pad1): track 4.39 -> 0.00 mm
- net Net-(D1-Pad2): track 0.00 -> 4.14 mm
- net Net-(J6-Pad2): track 22.5 -> 26.4 mm
- net +3V3: track 67.8 -> 71.7 mm, vias 19 -> 20
- net Net-(J67-Pad8): track 11.3 -> 12.4 mm
- net Net-(C8-Pad1): track 31.4 -> 30.5 mm
Other:
- board size 73.8 x 86.2 mm -> 73.8 x 89.6 mm

Commit message: update layout
Parts:
- removed J1: 3.3v, Connector_PinHeader_2.54mm:PinHeader_1x02_P2.54mm_Vertical
- moved J7 83.9 mm to (161.0, 102.5), turned to 180 degrees
- moved R13 78.8 mm to (152.4, 101.3)
- moved U5 74.9 mm to (159.4, 93.1), turned to 0 degrees
- moved D6 73.7 mm to (149.6, 101.3), turned to 90 degrees
- moved C9 63.8 mm to (150.2, 95.5), turned to 180 degrees
- moved C10 61.5 mm to (152.0, 88.7), turned to 90 degrees
- moved H2 23.1 mm to (161.0, 84.5)
- moved H3 22.4 mm to (112.0, 84.5)
- moved D1 16.3 mm to (121.8, 30.9), turned to 90 degrees
- moved R3 10.7 mm to (121.8, 36.9), turned to 270 degrees
- moved J70 8.81 mm to (162.2, 41.5), turned to 180 degrees
- moved J3 5.58 mm to (130.0, 83.5)
- moved J74 3.19 mm to (162.0, 48.2)
- moved H5 1.51 mm to (161.0, 26.5)
Routing:
- net Net-(J70-Pad2): track 0.00 -> 30.3 mm, vias 0 -> 1
- net Net-(J70-Pad1): track 0.00 -> 30.0 mm
- net /D9: track 25.6 -> 40.0 mm, vias 0 -> 2
- net /D13: track 13.5 -> 21.6 mm
- net Net-(J67-Pad8): track 12.4 -> 20.0 mm
- net Net-(J3-Pad9): track 16.1 -> 22.1 mm
- net Net-(J3-Pad11): track 18.4 -> 24.4 mm
- net Net-(J3-Pad12): track 20.3 -> 26.2 mm
- net /D12: track 20.4 -> 25.5 mm
- net Net-(J3-Pad5): track 11.9 -> 16.6 mm
- net Net-(J3-Pad4): track 17.8 -> 22.3 mm
- net Net-(J3-Pad7): track 14.6 -> 18.8 mm
- net Net-(J3-Pad10): track 18.0 -> 22.1 mm
- net Net-(J3-Pad8): track 16.5 -> 20.5 mm
- net Net-(J3-Pad6): track 14.7 -> 18.2 mm
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Other:
- board size 73.8 x 89.6 mm -> 56.5 x 86.2 mm

Commit message: update redesign
Parts:
- removed J4: Conn_02x04_Counter_Clockwise, Connector_PinHeader_2.54mm:PinHeader_2x04_P2.54mm_Vertical
- removed J71: Micro_SD_Card_Det, Connector_Card:microSD_HC_Hirose_DM3D-SF
- removed U2: samd51p20, Package_QFP:TQFP-128_14x14mm_P0.4mm
- added J1: Micro_SD_Card_Det, Connector_Card:microSD_HC_Hirose_DM3D-SF, F.Cu at (148.5, 30.4)
- added U1: samd51p20, Package_QFP:TQFP-128_14x14mm_P0.4mm, F.Cu at (136.9, 63.0)
- J3: value Conn_02x06_Counter_Clockwise -> Conn_02x16_Odd_Even; footprint Connector_PinHeader_2.54mm:PinHeader_2x06_P2.54mm_Vertical -> Connector_PinHeader_2.54mm:PinHeader_2x16_P2.54mm_Vertical
- moved J7 87.6 mm to (120.2, 25.0), turned to 270 degrees
- moved D6 78.5 mm to (111.5, 32.7)
- moved R13 76.6 mm to (111.5, 36.5), turned to 270 degrees
- moved U5 72.3 mm to (117.7, 34.0), turned to 90 degrees
- moved C10 61.1 mm to (113.4, 41.2), turned to 180 degrees
- moved C9 60.3 mm to (120.0, 43.3), turned to 270 degrees
- moved J3 23.8 mm to (150.4, 95.6)
- moved D1 4.44 mm to (125.4, 28.3)
- moved R3 4.44 mm to (125.4, 34.3)
- moved J74 0.25 mm to (161.7, 48.2)
Connections:
- J3 pad 1: GND -> +3V3
- J3 pad 3: Net-(J3-Pad3) -> +3V3
- J3 pad 4: Net-(J3-Pad4) -> GND
- J74 pad 1: +3V3 -> +5V
Routing:
- net Net-(J3-Pad19): track 0.00 -> 29.3 mm, vias 0 -> 1
- net Net-(J3-Pad22): track 0.00 -> 26.2 mm
- net Net-(J3-Pad24): track 0.00 -> 24.4 mm
- net Net-(J3-Pad11): track 24.4 -> 0.00 mm
- net Net-(J71-Pad3): track 24.3 -> 0.00 mm, vias 2 -> 0
- net Net-(J1-Pad3): track 0.00 -> 24.3 mm, vias 0 -> 2
- net Net-(J71-Pad5): track 23.2 -> 0.00 mm, vias 2 -> 0
- net Net-(J1-Pad5): track 0.00 -> 23.2 mm, vias 0 -> 2
- net Net-(J3-Pad4): track 22.3 -> 0.00 mm, vias 1 -> 0
- net Net-(J3-Pad9): track 22.1 -> 0.00 mm
- net Net-(J3-Pad28): track 0.00 -> 22.1 mm
- net Net-(J3-Pad26): track 0.00 -> 22.1 mm
- net Net-(J71-Pad8): track 21.2 -> 0.00 mm
- net Net-(J1-Pad8): track 0.00 -> 21.2 mm
- net Net-(J71-Pad7): track 21.2 -> 0.00 mm
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Other:
- board size 56.5 x 86.2 mm -> 56.5 x 65.5 mm

Commit message: update redesign
Parts:
- moved J3 13.7 mm to (155.6, 82.9)
Routing:
- net Net-(J3-Pad19): track 29.3 -> 15.2 mm, vias 1 -> 0
- net Net-(J3-Pad26): track 22.1 -> 11.2 mm
- net Net-(J3-Pad16): track 10.6 -> 0.00 mm
- net Net-(J3-Pad22): track 26.2 -> 16.1 mm
- net Net-(J3-Pad32): track 20.5 -> 10.7 mm
- net Net-(J3-Pad21): track 15.8 -> 7.38 mm, vias 1 -> 0
- net Net-(J3-Pad30): track 18.8 -> 11.1 mm
- net Net-(J3-Pad28): track 22.1 -> 14.5 mm
- net Net-(J3-Pad24): track 24.4 -> 17.8 mm
- net Net-(J3-Pad8): track 12.1 -> 8.51 mm
- net Net-(J3-Pad12): track 11.3 -> 7.80 mm
- net Net-(J3-Pad25): track 18.2 -> 15.1 mm
- net Net-(J3-Pad14): track 7.91 -> 6.39 mm
- net Net-(J3-Pad18): track 7.74 -> 6.54 mm

Commit message: update redesign
Parts:
- moved C16 1.25 mm to (137.2, 74.7)
- moved C18 0.60 mm to (139.2, 74.7)
Connections:
- J3 pad 1: +3V3 -> Net-(J3-Pad1)
- J3 pad 2: GND -> Net-(J3-Pad2)
- J3 pad 29: GND -> Net-(J3-Pad29)
- J3 pad 3: +3V3 -> Net-(J3-Pad3)
- J3 pad 31: GND -> Net-(J3-Pad31)
- J3 pad 4: GND -> Net-(J3-Pad4)
- U1 pad 27: Net-(J3-Pad24) -> Net-(J3-Pad31)
- U1 pad 28: Net-(J3-Pad22) -> Net-(J3-Pad29)
- U1 pad 29: Net-(J3-Pad28) -> Net-(J3-Pad27)
- U1 pad 30: Net-(J3-Pad26) -> Net-(J3-Pad25)
- U1 pad 33: Net-(J3-Pad30) -> Net-(J3-Pad23)
- U1 pad 34: Net-(J3-Pad32) -> Net-(J3-Pad21)
- U1 pad 35: Net-(J3-Pad27) -> Net-(J3-Pad19)
- U1 pad 36: Net-(J3-Pad25) -> Net-(J3-Pad17)
- U1 pad 37: Net-(J3-Pad23) -> +3V3
- U1 pad 39: Net-(J3-Pad21) -> Net-(J3-Pad15)
- U1 pad 40: Net-(J3-Pad19) -> Net-(J3-Pad13)
- U1 pad 41: Net-(J3-Pad17) -> Net-(J3-Pad11)
- U1 pad 42: Net-(J3-Pad15) -> Net-(J3-Pad9)
- U1 pad 43: Net-(J3-Pad13) -> Net-(J3-Pad7)
- U1 pad 44: Net-(J3-Pad11) -> Net-(J3-Pad5)
- U1 pad 47: Net-(J3-Pad9) -> Net-(U1-Pad47)
- U1 pad 48: Net-(J3-Pad7) -> Net-(U1-Pad48)
- U1 pad 49: Net-(J3-Pad5) -> Net-(U1-Pad49)
- U1 pad 56: Net-(J3-Pad20) -> Net-(J3-Pad16)
- U1 pad 57: Net-(J3-Pad18) -> Net-(J3-Pad14)
- U1 pad 58: Net-(J3-Pad16) -> Net-(J3-Pad12)
- U1 pad 59: Net-(J3-Pad14) -> Net-(J3-Pad10)
- U1 pad 60: Net-(J3-Pad12) -> Net-(J3-Pad8)
- U1 pad 61: Net-(J3-Pad10) -> Net-(J3-Pad6)
- U1 pad 62: Net-(J3-Pad8) -> Net-(J3-Pad4)
- U1 pad 63: Net-(J3-Pad6) -> Net-(J3-Pad2)
Routing:
- net Net-(J3-Pad5): track 0.00 -> 22.9 mm
- net Net-(J3-Pad31): track 0.00 -> 22.4 mm
- net Net-(J3-Pad7): track 0.00 -> 21.0 mm
- net Net-(J3-Pad29): track 0.00 -> 20.8 mm
- net Net-(J3-Pad9): track 0.00 -> 19.0 mm
- net Net-(J3-Pad24): track 17.8 -> 0.00 mm
- net Net-(J3-Pad11): track 0.00 -> 17.1 mm
- net Net-(J3-Pad22): track 16.1 -> 0.00 mm
- net Net-(J3-Pad17): track 0.00 -> 15.2 mm
- net Net-(J3-Pad13): track 0.00 -> 15.1 mm
- net Net-(J3-Pad28): track 14.5 -> 0.00 mm
- net Net-(J3-Pad15): track 0.00 -> 14.2 mm
- net Net-(J3-Pad23): track 0.00 -> 13.5 mm
- net Net-(J3-Pad26): track 11.2 -> 0.00 mm
- net Net-(J3-Pad30): track 11.1 -> 0.00 mm
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
Commit message: update
Parts:
- moved C19 0.30 mm to (149.2, 58.2)
Connections:
- J3 pad 1: Net-(J3-Pad1) -> +3V3
- J3 pad 18: Net-(J3-Pad18) -> GND
- J3 pad 20: Net-(J3-Pad20) -> GND
- J3 pad 22: Net-(J3-Pad22) -> GND
- J3 pad 24: Net-(J3-Pad24) -> GND
- J3 pad 26: Net-(J3-Pad26) -> GND
- J3 pad 28: Net-(J3-Pad28) -> GND
- J3 pad 3: Net-(J3-Pad3) -> +3V3
- J3 pad 30: Net-(J3-Pad30) -> GND
- J3 pad 32: Net-(J3-Pad32) -> GND
Routing:
- net Net-(J3-Pad2): track 2.91 -> 24.5 mm, vias 0 -> 1
- net Net-(J3-Pad4): track 3.27 -> 21.4 mm, vias 0 -> 1
- net Net-(J3-Pad12): track 0.00 -> 16.8 mm, vias 0 -> 1
- net Net-(J3-Pad6): track 4.65 -> 20.5 mm, vias 0 -> 1
- net Net-(J3-Pad16): track 0.00 -> 15.7 mm, vias 0 -> 1
- net Net-(J3-Pad8): track 4.97 -> 18.5 mm, vias 0 -> 1
- net Net-(J3-Pad10): track 6.39 -> 17.6 mm, vias 0 -> 1
- net Net-(J3-Pad14): track 5.59 -> 16.1 mm, vias 0 -> 1
- net +3V3: track 69.7 -> 77.4 mm, vias 18 -> 22
- net Net-(U1-Pad10): track 2.44 -> 0.00 mm, vias 1 -> 0
- added copper zone on B.Cu, net +3V3
Other:
- board text removed: "OSHW"
