File: electrosprawl.kicad_pcb (KiCad board)
At the start: 2 copper layers, 56.5 x 65.5 mm, 48 parts, among them J1 Micro_SD_Card_Det, J2 Conn_02x08_Counter_Clockwise, J3 Conn_02x16_Odd_Even, J5 Conn_02x08_Counter_Clockwise, J6 3.3v, J67 Conn_02x05_Counter_Clockwise, J7 VCC, J70 TXRX, J74 USB_B_Micro, SW1 Reset, U1 samd51p20, U5 LM1117-3.3, Y1 Crystal

Commit message: update
Parts:
- H4: footprint MountingHole:MountingHole_3mm -> MountingHole:MountingHole_3mm_Pad_Via
Connections:
- H4 pad 1: (no net) -> GND
Changed lines of the file:
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@@
     (add_net VCC)
+  )
+  (module MountingHole:MountingHole_3mm_Pad_Via (layer F.Cu)
+    (at 111.979434 26.482278 180)
+    (descr "Mounting Hole 3mm")
+    (tags "mounting hole 3mm")
+    (attr virtual)
+    (fp_text reference H4 (at 0 -4) (layer F.SilkS)
+      (effects (font (size 1 1) (thickness 0.15)))
+    )
+    (fp_text value MountingHole (at 0 4) (layer F.Fab)
+      (effects (font (size 1 1) (thickness 0.15)))
+    )
+    (fp_circle (center 0 0) (end 3.25 0) (layer F.CrtYd) (width 0.05))
+    (fp_circle (center 0 0) (end 3 0) (layer Cmts.User) (width 0.15))
+    (fp_text user %R (at 0.3 0) (layer F.Fab)
+      (effects (font (size 1 1) (thickness 0.15)))
+    )
+    (pad 1 thru_hole circle (at 1.59099 -1.59099 180) (size 0.8 0.8) (drill 0.5) (layers *.Cu *.Mask)
+      (net 2 GND))
+    (pad 1 thru_hole circle (at 0 -2.25 180) (size 0.8 0.8) (drill 0.5) (layers *.Cu *.Mask)
+      (net 2 GND))
+    (pad 1 thru_hole circle (at -1.59099 -1.59099 180) (size 0.8 0.8) (drill 0.5) (layers *.Cu *.Mask)
+      (net 2 GND))
+    (pad 1 thru_hole circle (at -2.25 0 180) (size 0.8 0.8) (drill 0.5) (layers *.Cu *.Mask)
+      (net 2 GND))
+    (pad 1 thru_hole circle (at -1.59099 1.59099 180) (size 0.8 0.8) (drill 0.5) (layers *.Cu *.Mask)
+      (net 2 GND))
+    (pad 1 thru_hole circle (at 0 2.25 180) (size 0.8 0.8) (drill 0.5) (layers *.Cu *.Mask)
+      (net 2 GND))
+    (pad 1 thru_hole circle (at 1.59099 1.59099 180) (size 0.8 0.8) (drill 0.5) (layers *.Cu *.Mask)
+      (net 2 GND))
+    (pad 1 thru_hole circle (at 2.25 0 180) (size 0.8 0.8) (drill 0.5) (layers *.Cu *.Mask)
+      (net 2 GND))
+    (pad 1 thru_hole circle (at 0 0 180) (size 6 6) (drill 3) (layers *.Cu *.Mask)
+      (net 2 GND))
   )
   (module Package_QFP:TQFP-128_14x14mm_P0.4mm (layer F.Cu)
@@
   )
   (module MountingHole:MountingHole_3mm (layer F.Cu)
-    (at 111.979434 26.482278 180)
-    (descr "Mounting Hole 3mm, no annular")
-    (tags "mounting hole 3mm no annular")
-    (attr virtual)
-    (fp_text reference H4 (at -2.286 0.0635 180) (layer F.SilkS)
-      (effects (font (size 0.5 0.5) (thickness 0.125)))
-    )
-    (fp_text value MountingHole (at 0 4 180) (layer F.Fab)
-      (effects (font (size 0.5 0.5) (thickness 0.125)))
-    )
-    (fp_circle (center 0 0) (end 3.25 0) (layer F.CrtYd) (width 0.05))
-    (fp_circle (center 0 0) (end 3 0) (layer Cmts.User) (width 0.15))
-    (fp_text user %R (at 0.3 0 180) (layer F.Fab)
-      (effects (font (size 1 1) (thickness 0.15)))
-    )
-    (pad 1 np_thru_hole circle (at 0 0 180) (size 3 3) (drill 3) (layers *.Cu *.Mask))
-  )
-  (module MountingHole:MountingHole_3mm (layer F.Cu)
