File: electrosprawl.sch (KiCad schematic (older format))
At the start: 123 parts, among them J1 3.3v, J10 A10, J11 A9, J12 A8, J13 A7, J14 A6, J15 A5, J16 A4, J17 A3, J18 A2, J19 reset, J2 D3, J20 D27, J21 D26, J22 D28, J23 Conn_01x04, J24 D23, J25 D22, J26 D12, J27 D11, J28 D10, J29 D9, J3 D2, J30 D8, J31 D7, J32 D6, J33 D5, J34 D4, J35 D44, J36 D43, J37 D42, J38 D41, J39 D40, J4 A15, J40 CAN, J41 I2C, J42 D37, J43 D36, J44 D35, J45 D34, J46 D33, J47 D32, J48 D31, J49 D30, J5 A14, J50 D29, J59 D49, J6 A13, J60 D48, J61 D47, J62 D46, J63 D45, J64 DAC, J65 AREF, J66 DAC, J67 Conn_02x05_Counter_Clockwise, J68 TXRX1CAN, J7 VCC, J70 TXRX, J71 Micro_SD_Card_Det, J73 I2C, J74 USB_B_Micro, J75 I2C, J76 I2C, J77 I2C, J78 I2C, J79 I2C, J8 A12, J80 I2C, J9 A11, SW1 Reset, U1 GD25Q32CTIGR, U2 samd51p20, U3 TCA9548APWR, U5 LM1117-3.3, Y1 Crystal

Commit message: update i2c with sx1509
Parts:
- removed C21: C_Small, Capacitor_SMD:C_0603_1608Metric, symbol Device:C_Small
- removed JP1, JP2, JP3: SolderJumper_2_Open, Jumper:SolderJumper-2_P1.3mm_Open_RoundedPad1.0x1.5mm, symbol Jumper:SolderJumper_2_Open
- removed R10, R11, R9: R10K, Resistor_SMD:R_0603_1608Metric, symbol Device:R
- removed U3: TCA9548APWR, Package_SO:TSSOP-24_4.4x7.8mm_P0.65mm, symbol Interface_Expansion:TCA9548APWR
- added J51, J52, J53, J54, J55, J56, J57, J58, J69, J72, J81, J82, J83, J84, J85, J86, J87, J88, J89, J90, J91, J92, J93, J94, J95, J96, J97: Conn_01x02, Connector_PinHeader_2.54mm:PinHeader_1x02_P2.54mm_Vertical, symbol Connector_Generic:Conn_01x02
- added U3, U4: SX1509, Package_DFN_QFN:QFN-28-1EP_4x4mm_P0.45mm_EP2.4x2.4mm, symbol SparkFun-DigitalIC:SX1509
- J19: value reset -> Conn_01x02
- J41, J73, J75, J76, J77, J78, J79, J80: value I2C -> Conn_01x02
Connections:
- wire segments 522 -> 713
Other:
- moved on the sheet: H2, H3, H4, H5, R12

Commit message: update layout redesign
Parts:
- removed J40: CAN, Connector_PinHeader_2.54mm:PinHeader_1x03_P2.54mm_Vertical, symbol Connector_Generic:Conn_01x03
- removed J68: TXRX1CAN, Connector_PinHeader_2.54mm:PinHeader_1x03_P2.54mm_Vertical, symbol Connector_Generic:Conn_01x03
- removed U1: GD25Q32CTIGR, GD25Q32CTIGR:SOIC127P600X175-8N, symbol GD25Q32CTIGR:GD25Q32CTIGR
- added J40, J68: Conn_01x02, Connector_PinHeader_2.54mm:PinHeader_1x02_P2.54mm_Vertical, symbol Connector_Generic:Conn_01x02
- J23: footprint Connector_PinHeader_2.54mm:PinHeader_1x04_P2.54mm_Vertical -> Connector_PinHeader_2.54mm:PinHeader_1x02_P2.54mm_Vertical
Connections:
- net labels removed: D38, D39
- wire segments 713 -> 681
Changed lines of the file:
@@
 	-1   0    0    1
 $EndComp
-$Comp
-L samd51p20:samd51p20 U2
-U 1 1 5C9E780D
-P 19300 9100
-F 0 "U2" H 20300 8800 50  0000 L CNN
-F 1 "samd51p20" H 19600 9100 50  0000 L CNN
-F 2 "Package_QFP:TQFP-128_14x14mm_P0.4mm" H 18800 10400 50  0001 C CNN
-F 3 "" H 18800 10400 50  0001 C CNN
-	1    19300 9100
-	1    0    0    -1
-$EndComp
 Wire Wire Line
 	21600 7550 21800 7550
@@
 	1    0    0    -1
 $EndComp
-$Comp
-L power:GND #PWR0127
-U 1 1 5CF96F26
-P 18300 14900
-F 0 "#PWR0127" H 18300 14650 50  0001 C CNN
-F 1 "GND" V 18305 14772 50  0000 R CNN
-F 2 "" H 18300 14900 50  0001 C CNN
-F 3 "" H 18300 14900 50  0001 C CNN
-	1    18300 14900
-	1    0    0    -1
-$EndComp
 Connection ~ 18750 3650
 Wire Wire Line
@@
 Wire Wire Line
 	19900 4600 19900 4800
-$Comp
-L power:+3.3V #PWR0128
-U 1 1 5D076B06
-P 18200 14400
-F 0 "#PWR0128" H 18200 14250 50  0001 C CNN
-F 1 "+3.3V" H 18215 14573 50  0000 C CNN
-F 2 "" H 18200 14400 50  0001 C CNN
-F 3 "" H 18200 14400 50  0001 C CNN
-	1    18200 14400
-	-1   0    0    1
-$EndComp
 Wire Wire Line
 	21600 7750 23000 7750
@@
 Wire Wire Line
 	18700 11150 18700 12350
-$Comp
-L Connector_Generic:Conn_01x03 J68
-U 1 1 5CEDF7BA
-P 18600 12550
-F 0 "J68" V 18473 12730 50  0000 L CNN
-F 1 "TXRX1CAN" V 18564 12730 50  0000 L CNN
-F 2 "Connector_PinHeader_2.54mm:PinHeader_1x03_P2.54mm_Vertical" H 18600 12550 50  0001 C CNN
-F 3 "~" H 18600 12550 50  0001 C CNN
-	1    18600 12550
-	0    1    1    0
-$EndComp
-Wire Wire Line
-	18300 11150 18300 11800
-Wire Wire Line
-	18500 11800 18500 12350
-Connection ~ 18300 11800
-Wire Wire Line
-	18300 11800 18500 11800
 Wire Wire Line
 	14850 9650 17100 9650
@@
 Text Label 21500 5850 0    50   ~ 0
 SDCD
-$Comp
-L GD25Q32CTIGR:GD25Q32CTIGR U1
-U 1 1 5D3B8472
-P 17350 13300
-F 0 "U1" V 17304 13930 50  0000 L CNN
-F 1 "GD25Q32CTIGR" V 17395 13930 50  0000 L CNN
-F 2 "GD25Q32CTIGR:SOIC127P600X175-8N" H 17350 13300 50  0001 L BNN
-F 3 "NOR FLASH" H 17350 13300 50  0001 L BNN
-F 4 "Unavailable" H 17350 13300 50  0001 L BNN "Field4"
-F 5 "None" H 17350 13300 50  0001 L BNN "Field5"
-F 6 "SOIC-8 GigaDevice Semiconductor _HK_ Limited" H 17350 13300 50  0001 L BNN "Field6"
-F 7 "GigaDevice Semiconductor _HK_ Limited" H 17350 13300 50  0001 L BNN "Field7"
-F 8 "GD25Q32CTIGR" H 17350 13300 50  0001 L BNN "Field8"
-	1    17350 13300
-	0    1    1    0
-$EndComp
-Wire Wire Line
-	17650 12800 17650 11550
-Wire Wire Line
-	17650 11550 18400 11550
-Wire Wire Line
-	18400 11550 18400 11150
-Wire Wire Line
-	17800 11150 17800 12650
-Wire Wire Line
-	17800 12650 17350 12650
-Wire Wire Line
-	17350 12650 17350 12800
-Wire Wire Line
-	18500 11150 18500 11500
-Wire Wire Line
-	18500 11500 17550 11500
-Wire Wire Line
-	17550 12800 17550 11500
-Wire Wire Line
-	18000 11150 18000 11450
-Wire Wire Line
-	17150 12800 17150 11450
-Wire Wire Line
-	17150 11450 18000 11450
-Wire Wire Line
-	18100 11150 18100 11400
-Wire Wire Line
-	18100 11400 17050 11400
-Wire Wire Line
-	17050 12800 17050 11400
-Wire Wire Line
-	17250 12800 17250 11350
-Wire Wire Line
-	17900 11350 17900 11150
-Wire Wire Line
-	17250 11350 17900 11350
-Wire Wire Line
-	18200 13950 17850 13950
-Wire Wire Line
-	18200 11150 18200 13950
-Wire Wire Line
-	17850 13800 17850 13950
-Wire Wire Line
-	18200 13950 18200 14400
-Connection ~ 18200 13950
-Wire Wire Line
-	18300 11800 18300 12850
-Wire Wire Line
-	16850 13800 16850 14100
-Wire Wire Line
-	16850 14100 18300 14100
-Wire Wire Line
-	18300 14100 18300 14900
-Connection ~ 18300 14100
 Wire Wire Line
 	18100 7050 18100 6850
@@
 Text Label 21900 10550 2    50   ~ 0
 D37
-Text Label 18900 11600 1    50   ~ 0
-D38
-Text Label 18800 11600 1    50   ~ 0
-D39
 Wire Wire Line
 	20200 11150 20200 11600
@@
 Wire Wire Line
 	14550 10550 14550 11100
-$Comp
-L Connector_Generic:Conn_01x03 J40
-U 1 1 5CAD745C
-P 18800 13150
-F 0 "J40" V 18673 13330 50  0000 L CNN
-F 1 "CAN" V 18764 13330 50  0000 L CNN
-F 2 "Connector_PinHeader_2.54mm:PinHeader_1x03_P2.54mm_Vertical" H 18800 13150 50  0001 C CNN
-F 3 "~" H 18800 13150 50  0001 C CNN
-	1    18800 13150
-	0    1    1    0
-$EndComp
 Wire Wire Line
 	18900 11150 18900 12950
 Wire Wire Line
 	18800 11150 18800 12950
-Wire Wire Line
-	18700 12950 18700 12850
-Wire Wire Line
-	18700 12850 18300 12850
-Connection ~ 18300 12850
-Wire Wire Line
-	18300 12850 18300 14100
 Connection ~ 10050 5250
 Connection ~ 10050 5600
@@
 F 0 "J23" V 19273 13180 50  0000 L CNN
 F 1 "Conn_01x04" V 19364 13180 50  0000 L CNN
-F 2 "Connector_PinHeader_2.54mm:PinHeader_1x04_P2.54mm_Vertical" H 19400 13000 50  0001 C CNN
+F 2 "Connector_PinHeader_2.54mm:PinHeader_1x02_P2.54mm_Vertical" H 19400 13000 50  0001 C CNN
 F 3 "~" H 19400 13000 50  0001 C CNN
 	1    19400 13000
@@
 	0    -1   -1   0
 $EndComp
+$Comp
+L Connector_Generic:Conn_01x02 J68
+U 1 1 5CC1A962
+P 18900 13150
+F 0 "J68" H 18980 13142 50  0000 L CNN
+F 1 "Conn_01x02" H 18980 13051 50  0000 L CNN
+F 2 "Connector_PinHeader_2.54mm:PinHeader_1x02_P2.54mm_Vertical" H 18900 13150 50  0001 C CNN
+F 3 "~" H 18900 13150 50  0001 C CNN
+	1    18900 13150
+	0    1    1    0
+$EndComp
+$Comp
+L Connector_Generic:Conn_01x02 J40
+U 1 1 5D7D70BD
+P 18700 12550
+F 0 "J40" H 18780 12542 50  0000 L CNN
+F 1 "Conn_01x02" H 18780 12451 50  0000 L CNN
+F 2 "Connector_PinHeader_2.54mm:PinHeader_1x02_P2.54mm_Vertical" H 18700 12550 50  0001 C CNN
+F 3 "~" H 18700 12550 50  0001 C CNN
+	1    18700 12550
+	0    1    1    0
+$EndComp
+$Comp
+L samd51p20:samd51p20 U2
+U 1 1 5C9E780D
+P 19300 9100
+F 0 "U2" H 20300 8800 50  0000 L CNN
+F 1 "samd51p20" H 19600 9100 50  0000 L CNN
+F 2 "Package_QFP:TQFP-128_14x14mm_P0.4mm" H 18800 10400 50  0001 C CNN
+F 3 "" H 18800 10400 50  0001 C CNN
+	1    19300 9100
+	1    0    0    -1
+$EndComp
 $EndSCHEMATC

Commit message: update layout
Parts:
- removed J19, J51: Conn_01x02, Connector_PinHeader_2.54mm:PinHeader_1x02_P2.54mm_Vertical, symbol Connector_Generic:Conn_01x02
- added C21, C24, C25: C_Small, Capacitor_SMD:C_0603_1608Metric, symbol Device:C_Small
- added R10, R9: R10K, Resistor_SMD:R_0603_1608Metric, symbol Device:R
- J23: footprint Connector_PinHeader_2.54mm:PinHeader_1x02_P2.54mm_Vertical -> Connector_PinHeader_2.54mm:PinHeader_1x04_P2.54mm_Vertical
- J32: value D6 -> Conn_01x02
Connections:
- net labels removed: D6
- wire segments 681 -> 682
- no-connect marks 0 -> 2
Changed lines of the file:
@@
 D7
-Wire Wire Line
-	21600 9150 21900 9150
-Text Label 21900 9150 2    50   ~ 0
-D6
 Wire Wire Line
 	21600 9650 21900 9650
@@
 D7
 $Comp
-L Connector_Generic:Conn_01x02 J32
-U 1 1 5DF95F32
-P 7800 9200
-F 0 "J32" H 7880 9192 50  0000 L CNN
-F 1 "D6" V 8100 8950 50  0000 L CNN
-F 2 "Connector_PinHeader_2.54mm:PinHeader_1x02_P2.54mm_Vertical" H 7800 9200 50  0001 C CNN
-F 3 "~" H 7800 9200 50  0001 C CNN
-	1    7800 9200
-	-1   0    0    1
-$EndComp
-Wire Wire Line
-	8000 9100 8200 9100
-Wire Wire Line
-	8000 9200 8550 9200
-Text Label 8550 9200 0    50   ~ 0
-D6
-$Comp
 L Connector_Generic:Conn_01x02 J33
 U 1 1 5DF95F3B
@@
 Wire Wire Line
 	8200 8750 8200 8400
-Connection ~ 8200 9100
-Wire Wire Line
-	8200 9100 8200 8750
 Connection ~ 8200 9450
-Wire Wire Line
-	8200 9450 8200 9100
 Wire Wire Line
 	11750 10550 11750 9800
@@
 Wire Wire Line
 	14550 10550 14550 11100
-Wire Wire Line
-	18900 11150 18900 12950
-Wire Wire Line
-	18800 11150 18800 12950
 Connection ~ 10050 5250
 Connection ~ 10050 5600
@@
 F 3 "~" H 22900 9750 50  0001 C CNN
 	1    22900 9750
-	-1   0    0    -1
+	-1   0    0    1
 $EndComp
 Wire Wire Line
@@
 F 0 "J23" V 19273 13180 50  0000 L CNN
 F 1 "Conn_01x04" V 19364 13180 50  0000 L CNN
-F 2 "Connector_PinHeader_2.54mm:PinHeader_1x02_P2.54mm_Vertical" H 19400 13000 50  0001 C CNN
+F 2 "Connector_PinHeader_2.54mm:PinHeader_1x04_P2.54mm_Vertical" H 19400 13000 50  0001 C CNN
 F 3 "~" H 19400 13000 50  0001 C CNN
 	1    19400 13000
@@
 	11750 3950 11750 8400
 Wire Wire Line
-	20900 11350 23200 11350
-$Comp
-L Connector_Generic:Conn_01x02 J19
-U 1 1 5D7EFDBE
-P 22850 10550
-F 0 "J19" H 22930 10542 50  0000 L CNN
-F 1 "Conn_01x02" H 22930 10451 50  0000 L CNN
-F 2 "Connector_PinHeader_2.54mm:PinHeader_1x02_P2.54mm_Vertical" H 22850 10550 50  0001 C CNN
-F 3 "~" H 22850 10550 50  0001 C CNN
-	1    22850 10550
-	-1   0    0    1
-$EndComp
-Wire Wire Line
 	22650 8750 22650 9250
 Connection ~ 22650 9250
 Wire Wire Line
 	22650 9250 22750 9250
-Wire Wire Line
-	23050 10450 23200 10450
-Wire Wire Line
-	23200 10450 23200 11350
 Wire Wire Line
 	24800 10900 24800 10850
@@
 $EndComp
 Wire Wire Line
-	24800 9250 25050 9250
-Wire Wire Line
-	23450 10250 23450 11350
-Wire Wire Line
-	23350 10250 23450 10250
-Connection ~ 23450 11350
-Connection ~ 23200 11350
-Wire Wire Line
-	23200 11350 23450 11350
-Wire Wire Line
 	23800 8750 22650 8750
-$Comp
-L Connector_Generic:Conn_01x02 J51
-U 1 1 5D5446E8
-P 23150 10350
-F 0 "J51" H 23230 10342 50  0000 L CNN
-F 1 "Conn_01x02" H 23230 10251 50  0000 L CNN
-F 2 "Connector_PinHeader_2.54mm:PinHeader_1x02_P2.54mm_Vertical" H 23150 10350 50  0001 C CNN
-F 3 "~" H 23150 10350 50  0001 C CNN
-	1    23150 10350
-	-1   0    0    1
-$EndComp
-Wire Wire Line
-	23050 10550 23800 10550
-Wire Wire Line
-	23350 10350 23800 10350
-Wire Wire Line
-	25050 8750 25050 9050
-Wire Wire Line
-	25050 9050 25050 9250
-Connection ~ 25050 9050
-Wire Wire Line
-	25250 9050 25050 9050
-Wire Wire Line
-	25250 10250 25250 9050
-Wire Wire Line
-	24800 10250 25250 10250
 Wire Wire Line
 	23800 8750 23800 8400
 Connection ~ 23800 8750
-Wire Wire Line
-	23800 8750 25050 8750
-Wire Wire Line
-	23800 9250 23800 8750
-Wire Wire Line
-	23450 11350 23550 11350
 Connection ~ 23550 11350
 Wire Wire Line
@@
 Connection ~ 23800 12450
 Wire Wire Line
-	23800 12450 25050 12450
-Wire Wire Line
-	23800 12950 23800 12450
+	23800 12450 24650 12450
+Wire Wire Line
+	23800 12950 23800 12750
 Wire Wire Line
 	23650 15050 23800 15050
@@
 	20900 11150 20900 11350
 Wire Wire Line
-	20900 15050 20900 11350
+	20900 15050 20900 14050
 Connection ~ 20900 11350
 Wire Wire Line
@@
 $EndComp
 $Comp
-L Connector_Generic:Conn_01x02 J68
-U 1 1 5CC1A962
-P 18900 13150
-F 0 "J68" H 18980 13142 50  0000 L CNN
-F 1 "Conn_01x02" H 18980 13051 50  0000 L CNN
-F 2 "Connector_PinHeader_2.54mm:PinHeader_1x02_P2.54mm_Vertical" H 18900 13150 50  0001 C CNN
-F 3 "~" H 18900 13150 50  0001 C CNN
-	1    18900 13150
-	0    1    1    0
-$EndComp
-$Comp
 L Connector_Generic:Conn_01x02 J40
 U 1 1 5D7D70BD
@@
 	1    0    0    -1
 $EndComp
+$Comp
+L Connector_Generic:Conn_01x02 J68
+U 1 1 5D4BCA69
+P 22350 8450
+F 0 "J68" H 22430 8442 50  0000 L CNN
+F 1 "Conn_01x02" H 22430 8351 50  0000 L CNN
+F 2 "Connector_PinHeader_2.54mm:PinHeader_1x02_P2.54mm_Vertical" H 22350 8450 50  0001 C CNN
+F 3 "~" H 22350 8450 50  0001 C CNN
+	1    22350 8450
+	1    0    0    -1
+$EndComp
+Wire Wire Line
+	21600 8450 22150 8450
+Wire Wire Line
+	21600 8550 22150 8550
+$Comp
+L Connector_Generic:Conn_01x02 J32
+U 1 1 5DB2E53F
+P 17800 11850
+F 0 "J32" H 17880 11842 50  0000 L CNN
+F 1 "Conn_01x02" H 17880 11751 50  0000 L CNN
+F 2 "Connector_PinHeader_2.54mm:PinHeader_1x02_P2.54mm_Vertical" H 17800 11850 50  0001 C CNN
+F 3 "~" H 17800 11850 50  0001 C CNN
+	1    17800 11850
+	0    1    1    0
+$EndComp
+Wire Wire Line
+	17800 11650 17800 11150
+$Comp
+L power:GND #PWR0125
+U 1 1 5E183F27
+P 17700 11450
+F 0 "#PWR0125" H 17700 11200 50  0001 C CNN
+F 1 "GND" V 17705 11322 50  0000 R CNN
+F 2 "" H 17700 11450 50  0001 C CNN
+F 3 "" H 17700 11450 50  0001 C CNN
+	1    17700 11450
+	-1   0    0    1
+$EndComp
+Wire Wire Line
+	17700 11450 17700 11650
+Wire Wire Line
+	8200 8750 8200 9450
+Wire Wire Line
+	23800 9250 23800 9050
+Wire Wire Line
+	23650 9850 23800 9850
+$Comp
+L Device:R R10
+U 1 1 5D03240C
+P 23650 9500
+F 0 "R10" V 23443 9500 50  0000 C CNN
+F 1 "R10K" V 23534 9500 50  0000 C CNN
+F 2 "Resistor_SMD:R_0603_1608Metric" V 23580 9500 50  0001 C CNN
+F 3 "~" H 23650 9500 50  0001 C CNN
+	1    23650 9500
+	-1   0    0    1
+$EndComp
+Wire Wire Line
+	23650 9650 23650 9850
+Wire Wire Line
+	23800 9050 23650 9050
+Wire Wire Line
+	23650 9050 23650 9350
+Connection ~ 23800 9050
+Wire Wire Line
+	23800 9050 23800 8750
+Wire Wire Line
+	23600 13350 23600 13550
+Wire Wire Line
+	23600 13550 23800 13550
+$Comp
+L Device:R R9
+U 1 1 5D705667
+P 23600 13200
+F 0 "R9" V 23393 13200 50  0000 C CNN
+F 1 "R10K" V 23484 13200 50  0000 C CNN
+F 2 "Resistor_SMD:R_0603_1608Metric" V 23530 13200 50  0001 C CNN
+F 3 "~" H 23600 13200 50  0001 C CNN
+	1    23600 13200
+	-1   0    0    1
+$EndComp
+Wire Wire Line
+	23800 12750 23600 12750
+Wire Wire Line
+	23600 12750 23600 13050
+Connection ~ 23800 12750
+Wire Wire Line
+	23800 12750 23800 12450
+$Comp
+L Device:C_Small C21
+U 1 1 5DA4452B
+P 16200 10300
+F 0 "C21" H 16292 10346 50  0000 L CNN
+F 1 "C_Small" H 16292 10255 50  0000 L CNN
+F 2 "Capacitor_SMD:C_0603_1608Metric" H 16200 10300 50  0001 C CNN
+F 3 "~" H 16200 10300 50  0001 C CNN
+	1    16200 10300
+	-1   0    0    1
+$EndComp
+Connection ~ 16200 10400
+Connection ~ 16200 10200
+$Comp
+L Device:C_Small C25
+U 1 1 5DA4BD02
+P 24850 12350
+F 0 "C25" H 24942 12396 50  0000 L CNN
+F 1 "C_Small" H 24942 12305 50  0000 L CNN
+F 2 "Capacitor_SMD:C_0603_1608Metric" H 24850 12350 50  0001 C CNN
+F 3 "~" H 24850 12350 50  0001 C CNN
+	1    24850 12350
+	-1   0    0    1
+$EndComp
+Connection ~ 24850 12450
+Wire Wire Line
+	24850 12450 25050 12450
+$Comp
+L Device:C_Small C24
+U 1 1 5DAC483F
+P 24650 12350
+F 0 "C24" H 24742 12396 50  0000 L CNN
+F 1 "C_Small" H 24742 12305 50  0000 L CNN
+F 2 "Capacitor_SMD:C_0603_1608Metric" H 24650 12350 50  0001 C CNN
+F 3 "~" H 24650 12350 50  0001 C CNN
+	1    24650 12350
+	-1   0    0    1
+$EndComp
+Connection ~ 24650 12450
+Wire Wire Line
+	24650 12450 24850 12450
+Wire Wire Line
+	23800 11350 24250 11350
+Connection ~ 23800 11350
+Wire Wire Line
+	24250 12250 24650 12250
+Wire Wire Line
+	24250 11350 24250 12250
+Connection ~ 24650 12250
+Wire Wire Line
+	24650 12250 24850 12250
+Wire Wire Line
+	20450 14050 20900 14050
+Connection ~ 20900 14050
+Wire Wire Line
+	20900 14050 20900 11350
+$Comp
+L power:GND #PWR0128
+U 1 1 5EBDE98B
+P 20450 14050
+F 0 "#PWR0128" H 20450 13800 50  0001 C CNN
+F 1 "GND" V 20455 13922 50  0000 R CNN
+F 2 "" H 20450 14050 50  0001 C CNN
+F 3 "" H 20450 14050 50  0001 C CNN
+	1    20450 14050
+	0    1    1    0
+$EndComp
+NoConn ~ 24800 9250
+NoConn ~ 24800 10250
+Wire Wire Line
+	20900 11350 23550 11350
 $EndSCHEMATC

Commit message: update layout
Parts:
- removed C21, C24, C25: C_Small, Capacitor_SMD:C_0603_1608Metric, symbol Device:C_Small
- removed J41, J52, J73, J75, J76, J77, J78, J79, J80, J81, J82, J83, J90, J91, J92, J93, J94, J95, J96, J97: Conn_01x02, Connector_PinHeader_2.54mm:PinHeader_1x02_P2.54mm_Vertical, symbol Connector_Generic:Conn_01x02
- removed R12, R9: R10K, Resistor_SMD:R_0603_1608Metric, symbol Device:R
- removed U4: SX1509, Package_DFN_QFN:QFN-28-1EP_4x4mm_P0.45mm_EP2.4x2.4mm, symbol SparkFun-DigitalIC:SX1509
Connections:
- wire segments 682 -> 538
- no-connect marks 2 -> 26

Commit message: update redesign
Parts:
- removed J10: A10, Connector_PinHeader_2.54mm:PinHeader_1x02_P2.54mm_Vertical, symbol Connector_Generic:Conn_01x02
- removed J11: A9, Connector_PinHeader_2.54mm:PinHeader_1x02_P2.54mm_Vertical, symbol Connector_Generic:Conn_01x02
- removed J12: A8, Connector_PinHeader_2.54mm:PinHeader_1x02_P2.54mm_Vertical, symbol Connector_Generic:Conn_01x02
- removed J13: A7, Connector_PinHeader_2.54mm:PinHeader_1x02_P2.54mm_Vertical, symbol Connector_Generic:Conn_01x02
- removed J14: A6, Connector_PinHeader_2.54mm:PinHeader_1x02_P2.54mm_Vertical, symbol Connector_Generic:Conn_01x02
- removed J15: A5, Connector_PinHeader_2.54mm:PinHeader_1x02_P2.54mm_Vertical, symbol Connector_Generic:Conn_01x02
- removed J16: A4, Connector_PinHeader_2.54mm:PinHeader_1x02_P2.54mm_Vertical, symbol Connector_Generic:Conn_01x02
- removed J17: A3, Connector_PinHeader_2.54mm:PinHeader_1x02_P2.54mm_Vertical, symbol Connector_Generic:Conn_01x02
- removed J18: A2, Connector_PinHeader_2.54mm:PinHeader_1x02_P2.54mm_Vertical, symbol Connector_Generic:Conn_01x02
- removed J2: D3, Connector_PinHeader_2.54mm:PinHeader_1x02_P2.54mm_Vertical, symbol Connector_Generic:Conn_01x02
- removed J20: D27, Connector_PinHeader_2.54mm:PinHeader_1x02_P2.54mm_Vertical, symbol Connector_Generic:Conn_01x02
- removed J21: D26, Connector_PinHeader_2.54mm:PinHeader_1x02_P2.54mm_Vertical, symbol Connector_Generic:Conn_01x02
- removed J22: D28, Connector_PinHeader_2.54mm:PinHeader_1x02_P2.54mm_Vertical, symbol Connector_Generic:Conn_01x02
- removed J24: D23, Connector_PinHeader_2.54mm:PinHeader_1x02_P2.54mm_Vertical, symbol Connector_Generic:Conn_01x02
- removed J25: D22, Connector_PinHeader_2.54mm:PinHeader_1x02_P2.54mm_Vertical, symbol Connector_Generic:Conn_01x02
- removed J3: D2, Connector_PinHeader_2.54mm:PinHeader_1x02_P2.54mm_Vertical, symbol Connector_Generic:Conn_01x02
- removed J30: D8, Connector_PinHeader_2.54mm:PinHeader_1x02_P2.54mm_Vertical, symbol Connector_Generic:Conn_01x02
- removed J31: D7, Connector_PinHeader_2.54mm:PinHeader_1x02_P2.54mm_Vertical, symbol Connector_Generic:Conn_01x02
- removed J33: D5, Connector_PinHeader_2.54mm:PinHeader_1x02_P2.54mm_Vertical, symbol Connector_Generic:Conn_01x02
- removed J34: D4, Connector_PinHeader_2.54mm:PinHeader_1x02_P2.54mm_Vertical, symbol Connector_Generic:Conn_01x02
- removed J35: D44, Connector_PinHeader_2.54mm:PinHeader_1x02_P2.54mm_Vertical, symbol Connector_Generic:Conn_01x02
- removed J36: D43, Connector_PinHeader_2.54mm:PinHeader_1x02_P2.54mm_Vertical, symbol Connector_Generic:Conn_01x02
- removed J37: D42, Connector_PinHeader_2.54mm:PinHeader_1x02_P2.54mm_Vertical, symbol Connector_Generic:Conn_01x02
- removed J38: D41, Connector_PinHeader_2.54mm:PinHeader_1x02_P2.54mm_Vertical, symbol Connector_Generic:Conn_01x02
- removed J39: D40, Connector_PinHeader_2.54mm:PinHeader_1x02_P2.54mm_Vertical, symbol Connector_Generic:Conn_01x02
- removed J4: A15, Connector_PinHeader_2.54mm:PinHeader_1x02_P2.54mm_Vertical, symbol Connector_Generic:Conn_01x02
- removed J42: D37, Connector_PinHeader_2.54mm:PinHeader_1x02_P2.54mm_Vertical, symbol Connector_Generic:Conn_01x02
- removed J43: D36, Connector_PinHeader_2.54mm:PinHeader_1x02_P2.54mm_Vertical, symbol Connector_Generic:Conn_01x02
- removed J44: D35, Connector_PinHeader_2.54mm:PinHeader_1x02_P2.54mm_Vertical, symbol Connector_Generic:Conn_01x02
- removed J45: D34, Connector_PinHeader_2.54mm:PinHeader_1x02_P2.54mm_Vertical, symbol Connector_Generic:Conn_01x02
- removed J46: D33, Connector_PinHeader_2.54mm:PinHeader_1x02_P2.54mm_Vertical, symbol Connector_Generic:Conn_01x02
- removed J47: D32, Connector_PinHeader_2.54mm:PinHeader_1x02_P2.54mm_Vertical, symbol Connector_Generic:Conn_01x02
- removed J48: D31, Connector_PinHeader_2.54mm:PinHeader_1x02_P2.54mm_Vertical, symbol Connector_Generic:Conn_01x02
- removed J49: D30, Connector_PinHeader_2.54mm:PinHeader_1x02_P2.54mm_Vertical, symbol Connector_Generic:Conn_01x02
- removed J5: A14, Connector_PinHeader_2.54mm:PinHeader_1x02_P2.54mm_Vertical, symbol Connector_Generic:Conn_01x02
- removed J50: D29, Connector_PinHeader_2.54mm:PinHeader_1x02_P2.54mm_Vertical, symbol Connector_Generic:Conn_01x02
- removed J59: D49, Connector_PinHeader_2.54mm:PinHeader_1x02_P2.54mm_Vertical, symbol Connector_Generic:Conn_01x02
- removed J6: A13, Connector_PinHeader_2.54mm:PinHeader_1x02_P2.54mm_Vertical, symbol Connector_Generic:Conn_01x02
- removed J60: D48, Connector_PinHeader_2.54mm:PinHeader_1x02_P2.54mm_Vertical, symbol Connector_Generic:Conn_01x02
- removed J61: D47, Connector_PinHeader_2.54mm:PinHeader_1x02_P2.54mm_Vertical, symbol Connector_Generic:Conn_01x02
- removed J62: D46, Connector_PinHeader_2.54mm:PinHeader_1x02_P2.54mm_Vertical, symbol Connector_Generic:Conn_01x02
- removed J63: D45, Connector_PinHeader_2.54mm:PinHeader_1x02_P2.54mm_Vertical, symbol Connector_Generic:Conn_01x02
- removed J8: A12, Connector_PinHeader_2.54mm:PinHeader_1x02_P2.54mm_Vertical, symbol Connector_Generic:Conn_01x02
- removed J9: A11, Connector_PinHeader_2.54mm:PinHeader_1x02_P2.54mm_Vertical, symbol Connector_Generic:Conn_01x02
- added J2, J?: Conn_02x08_Odd_Even, Connector_PinHeader_2.54mm:PinHeader_2x08_P2.54mm_Vertical, symbol Connector_Generic:Conn_02x08_Odd_Even
- U2: symbol samd51p20:samd51p20 -> electrosprawl-rescue:samd51p20-samd51p20
Connections:
- wire segments 538 -> 432
